Commit message: Created new package trailer_controller and yaml file

File: install/trailer_description/share/trailer_description/urdf/trailer_gazebo.xacro (robot description, xacro)
@@ -1,4 +1,18 @@
 <?xml version="1.0" encoding="utf-8"?>
 <robot name="trailer" xmlns:xacro="http://www.ros.org/wiki/xacro">
+    <transmission name="left_wheel_transmission">
+        <plugin>transmission_interface/SimpleTransmission</plugin>
+        <actuator name="left_wheel_motor" role="actuator_left"/>
+        <joint name="b_back_left_wheel_joint" role="joint_left">
+            <mechanicalReduction>1.0</mechanicalReduction>
+        </joint>
+    </transmission>
+    <transmission name="right_wheel_transmission">
+        <plugin>transmission_interface/SimpleTransmission</plugin>
+        <actuator name="right_wheel_motor" role="actuator_right"/>
+        <joint name="b_back_right_wheel_joint" role="joint_right">
+            <mechanicalReduction>1.0</mechanicalReduction>
+        </joint>
+    </transmission>
     <gazebo reference="b_front_left_wheel">
         <mu1>100000000000000.0</mu1>
@@ -55,3 +69,10 @@
         <fdir1>0 -1 0</fdir1>
     </gazebo>
+    <gazebo>
+        <plugin filename="libgazebo_ros2_control.so" name="gazebo_ros2_control">
+            <robot_param>robot_description</robot_param>
+            <robot_param_node>robot_state_publisher</robot_param_node>
+            <parameters>find trailer_controller/config/trailer_controller.yaml</parameters>
+        </plugin>
+    </gazebo>
 </robot>

File: src/trailer_description/urdf/trailer_gazebo.xacro (robot description, xacro)
@@ -73,5 +73,5 @@
             <robot_param>robot_description</robot_param>
             <robot_param_node>robot_state_publisher</robot_param_node>
-            <parameters></parameters>
+            <parameters>find trailer_controller/config/trailer_controller.yaml</parameters>
         </plugin>
     </gazebo>

Commit message: .

File: install/trailer_description/share/trailer_description/urdf/trailer_gazebo.xacro (robot description, xacro)
@@ -12,4 +12,18 @@
         <actuator name="right_wheel_motor" role="actuator_right"/>
         <joint name="b_back_right_wheel_joint" role="joint_right">
+            <mechanicalReduction>1.0</mechanicalReduction>
+        </joint>
+    </transmission>
+    <transmission name="left_linkage_transmission">
+        <plugin>transmission_interface/SimpleTransmission</plugin>
+        <actuator name="left_linkage_actuator" role="actuator_left"/>
+        <joint name="b_front_left_linkage_joint" role="joint_left">
+            <mechanicalReduction>1.0</mechanicalReduction>
+        </joint>
+    </transmission>
+    <transmission name="right_linkage_transmission">
+        <plugin>transmission_interface/SimpleTransmission</plugin>
+        <actuator name="right_linkage_actuator" role="actuator_right"/>
+        <joint name="b_front_right_linkage_joint" role="joint_right">
             <mechanicalReduction>1.0</mechanicalReduction>
         </joint>
@@ -73,5 +87,5 @@
             <robot_param>robot_description</robot_param>
             <robot_param_node>robot_state_publisher</robot_param_node>
-            <parameters>find trailer_controller/config/trailer_controller.yaml</parameters>
+            <parameters>$(find trailer_controller)/config/trailer_controller.yaml</parameters>
         </plugin>
     </gazebo>

File: install/trailer_description/share/trailer_description/urdf/trailer_ros2_control.xacro (robot description, xacro)
@@ -5,5 +5,6 @@
             <plugin>gazebo_ros2_control/GazeboSystem</plugin>
         </hardware>
-        <joint name="left_wheel_transmission">
+        <!-- Back wheel joints -->
+        <joint name="b_back_left_wheel_joint">
             <command_interface name="velocity">
                 <param name="min">-1</param>
@@ -13,5 +14,5 @@
             <state_interface name="velocity"/>
         </joint>
-        <joint name="right_wheel_transmission">
+        <joint name="b_back_right_wheel_joint">
             <command_interface name="velocity">
                 <param name="min">-1</param>
@@ -21,4 +22,21 @@
             <state_interface name="velocity"/>
         </joint>
+        <!-- Steering linkage joints -->
+        <joint name="b_front_left_linkage_joint">
+            <command_interface name="position">
+                <param name="min">-0.5</param>
+                <param name="max">0.5</param>
+            </command_interface>
+            <state_interface name="position"/>
+            <state_interface name="velocity"/>
+        </joint>
+        <joint name="b_front_right_linkage_joint">
+            <command_interface name="position">
+                <param name="min">-0.5</param>
+                <param name="max">0.5</param>
+            </command_interface>
+            <state_interface name="position"/>
+            <state_interface name="velocity"/>
+        </joint>
     </ros2_control>
 </robot>

Commit message: I was able to control the steering and the entire truck-trailer were working, including all tyres.

File: install/trailer_description/share/trailer_description/urdf/trailer_gazebo.xacro (robot description, xacro)
@@ -18,6 +18,6 @@
         <plugin>transmission_interface/SimpleTransmission</plugin>
         <actuator name="left_steer_actuator" role="actuator_left"/>
-        <joint name="steer_left_joint" role="joint_left">
-            <mechanicalReduction>1.0</mechanicalReduction>
+        <joint name="steer_left_joint" role="joint_left_steer">
+            <mechanicalReduction>25.13276</mechanicalReduction>
         </joint>
     </transmission>
@@ -25,8 +25,26 @@
         <plugin>transmission_interface/SimpleTransmission</plugin>
         <actuator name="right_steer_actuator" role="actuator_right"/>
-        <joint name="steer_right_joint" role="joint_right">
-            <mechanicalReduction>1.0</mechanicalReduction>
+        <joint name="steer_right_joint" role="joint_right_steer">
+            <mechanicalReduction>25.13276</mechanicalReduction>
         </joint>
     </transmission>
+    <gazebo reference="steer_left">
+        <mu1>1.0</mu1>
+        <mu2>1.0</mu2>
+        <kp>50000.0</kp>
+        <kd>50.0</kd>
+        <minDepth>0.001</minDepth>
+        <maxVel>0.1</maxVel>
+        <fdir1>0 -1 0</fdir1>
+    </gazebo>
+    <gazebo reference="steer_right">
+        <mu1>1.0</mu1>
+        <mu2>1.0</mu2>
+        <kp>50000.0</kp>
+        <kd>50.0</kd>
+        <minDepth>0.001</minDepth>
+        <maxVel>0.1</maxVel>
+        <fdir1>0 1 0</fdir1>
+    </gazebo>
     <gazebo reference="front_left_wheel">
         <mu1>100000000000000.0</mu1>
@@ -92,5 +110,5 @@
         <fdir1>0 -1 0</fdir1>
     </gazebo>
-    <!-- <gazebo>
+    <gazebo>
         <plugin filename="libgazebo_ros2_control.so" name="gazebo_ros2_control">
             <robot_param>robot_description</robot_param>
@@ -98,4 +116,9 @@
             <parameters>$(find trailer_controller)/config/trailer_controller.yaml</parameters>
         </plugin>
+    </gazebo>
+    <!-- <gazebo>
+        <plugin filename="libgazebo_ros2_control.so" name="gazebo_ros2_control">
+            <parameters>$(find trailer_controller)/config/ackermann_steering_controller_params.yaml</parameters>
+        </plugin>
     </gazebo> -->
 </robot>

File: install/trailer_description/share/trailer_description/urdf/trailer_ros2_control.xacro (robot description, xacro)
@@ -5,5 +5,5 @@
             <plugin>gazebo_ros2_control/GazeboSystem</plugin>
         </hardware>
-        <!-- Back wheel joints -->
+        <!-- Rear wheel joints -->
         <joint name="rear_left_wheel_joint">
             <command_interface name="velocity">
@@ -40,8 +40,8 @@
         </joint>
     </ros2_control>
-    <gazebo>
+    <!-- <gazebo>
         <plugin filename="libgazebo_ros2_control.so" name="gazebo_ros2_control">
             <parameters>$(find trailer_controller)/config/ackermann_steering_controller_params.yaml</parameters>
         </plugin>
-    </gazebo>
+    </gazebo> -->
 </robot>

File: src/trailer_description/urdf/trailer_gazebo.xacro (robot description, xacro)
@@ -18,6 +18,6 @@
         <plugin>transmission_interface/SimpleTransmission</plugin>
         <actuator name="left_steer_actuator" role="actuator_left"/>
-        <joint name="steer_left_joint" role="joint_left">
-            <mechanicalReduction>1.0</mechanicalReduction>
+        <joint name="steer_left_joint" role="joint_left_steer">
+            <mechanicalReduction>25.13276</mechanicalReduction>
         </joint>
     </transmission>
@@ -25,6 +25,6 @@
         <plugin>transmission_interface/SimpleTransmission</plugin>
         <actuator name="right_steer_actuator" role="actuator_right"/>
-        <joint name="steer_right_joint" role="joint_right">
-            <mechanicalReduction>1.0</mechanicalReduction>
+        <joint name="steer_right_joint" role="joint_right_steer">
+            <mechanicalReduction>25.13276</mechanicalReduction>
         </joint>
     </transmission>
@@ -110,5 +110,5 @@
         <fdir1>0 -1 0</fdir1>
     </gazebo>
-    <!-- <gazebo>
+    <gazebo>
         <plugin filename="libgazebo_ros2_control.so" name="gazebo_ros2_control">
             <robot_param>robot_description</robot_param>
@@ -116,4 +116,9 @@
             <parameters>$(find trailer_controller)/config/trailer_controller.yaml</parameters>
         </plugin>
+    </gazebo>
+    <!-- <gazebo>
+        <plugin filename="libgazebo_ros2_control.so" name="gazebo_ros2_control">
+            <parameters>$(find trailer_controller)/config/ackermann_steering_controller_params.yaml</parameters>
+        </plugin>
     </gazebo> -->
 </robot>
