Commit message: .

File: install/trailer_description/share/trailer_description/urdf/trailer.urdf.xacro (robot description, xacro)
@@ -10,15 +10,15 @@
     <inertial>
       <origin
-        xyz="0.01453437491039 -4.90378546530802E-11 0.504525903309878"
+        xyz="0.0145343749103901 -4.8067090025433E-11 0.504525903309878"
         rpy="0 0 0" />
       <mass
         value="5621.45261479066" />
       <inertia
-        ixx="1504.40687433883"
-        ixy="6.00339758754412E-07"
+        ixx="1504.39932306857"
+        ixy="5.67577165358734E-07"
         ixz="-97.6855056473575"
         iyy="7926.87309013488"
-        iyz="-6.53887552382793E-08"
-        izz="8441.85088000873" />
+        iyz="-6.11751972034413E-08"
+        izz="8441.84332873847" />
     </inertial>
     <visual>
@@ -52,53 +52,53 @@
   </joint>
   <link
-    name="b_front_left_linkage">
-    <inertial>
-      <origin
-        xyz="2.01833247004402E-07 0.0866174322359835 0.114144894811921"
-        rpy="0 0 0" />
-      <mass
-        value="4.04562727792635" />
-      <inertia
-        ixx="0.140037164042004"
-        ixy="5.5743582115057E-08"
-        ixz="-2.0885090231136E-08"
-        iyy="0.0827902917589038"
-        iyz="0.0400096165626046"
-        izz="0.0604906292211793" />
-    </inertial>
-    <visual>
-      <origin
-        xyz="0 0 0"
-        rpy="0 0 0" />
-      <geometry>
-        <mesh
-          filename="package://trailer_description/meshes/b_front_left_linkage.STL" />
-      </geometry>
-      <material
-        name="">
-        <color
-          rgba="0.792156862745098 0.819607843137255 0.933333333333333 1" />
-      </material>
-    </visual>
-    <collision>
-      <origin
-        xyz="0 0 0"
-        rpy="0 0 0" />
-      <geometry>
-        <mesh
-          filename="package://trailer_description/meshes/b_front_left_linkage.STL" />
-      </geometry>
-    </collision>
-  </link>
-  <joint
-    name="b_front_left_linkage_joint"
+    name="left_linkage">
+    <inertial>
+      <origin
+        xyz="2.01833246560312E-07 0.086617432235983 0.114144894811922"
+        rpy="0 0 0" />
+      <mass
+        value="4.04562727792638" />
+      <inertia
+        ixx="0.140037164042005"
+        ixy="5.57435821298368E-08"
+        ixz="-2.08850902365895E-08"
+        iyy="0.0827902917589043"
+        iyz="0.0400096165626049"
+        izz="0.0604906292211796" />
+    </inertial>
+    <visual>
+      <origin
+        xyz="0 0 0"
+        rpy="0 0 0" />
+      <geometry>
+        <mesh
+          filename="package://trailer_description/meshes/left_linkage.STL" />
+      </geometry>
+      <material
+        name="">
+        <color
+          rgba="0.792156862745098 0.819607843137255 0.933333333333333 1" />
+      </material>
+    </visual>
+    <collision>
+      <origin
+        xyz="0 0 0"
+        rpy="0 0 0" />
+      <geometry>
+        <mesh
+          filename="package://trailer_description/meshes/left_linkage.STL" />
+      </geometry>
+    </collision>
+  </link>
+  <joint
+    name="left_linkage_joint"
     type="revolute">
     <origin
-      xyz="1.46 0.3625 0"
+      xyz="1.46 0.385 0"
       rpy="0 0 0" />
     <parent
       link="base_link" />
     <child
-      link="b_front_left_linkage" />
+      link="left_linkage" />
     <axis
       xyz="0 0 1" />
@@ -110,5 +110,5 @@
   </joint>
   <link
-    name="b_front_left_wheel">
+    name="front_left_wheel">
     <inertial>
       <origin
@@ -131,24 +131,24 @@
       <geometry>
         <mesh
-          filename="package://trailer_description/meshes/b_front_left_wheel.STL" />
-      </geometry>
-      <material
-        name="">
-        <color
-          rgba="0.792156862745098 0.819607843137255 0.933333333333333 1" />
-      </material>
-    </visual>
-    <collision>
-      <origin
-        xyz="0 0 0"
-        rpy="0 0 0" />
-      <geometry>
-        <mesh
-          filename="package://trailer_description/meshes/b_front_left_wheel.STL" />
-      </geometry>
-    </collision>
-  </link>
-  <joint
-    name="b_front_left_wheel_joint"
+          filename="package://trailer_description/meshes/front_left_wheel.STL" />
+      </geometry>
+      <material
+        name="">
+        <color
+          rgba="0.792156862745098 0.819607843137255 0.933333333333333 1" />
+      </material>
+    </visual>
+    <collision>
+      <origin
+        xyz="0 0 0"
+        rpy="0 0 0" />
+      <geometry>
+        <mesh
+          filename="package://trailer_description/meshes/front_left_wheel.STL" />
+      </geometry>
+    </collision>
+  </link>
+  <joint
+    name="front_left_wheel_joint"
     type="continuous">
     <origin
@@ -156,7 +156,7 @@
       rpy="0 0 0" />
     <parent
-      link="b_front_left_linkage" />
-    <child
-      link="b_front_left_wheel" />
+      link="left_linkage" />
+    <child
+      link="front_left_wheel" />
     <axis
       xyz="0 -1 0" />
@@ -166,53 +166,53 @@
   </joint>
   <link
-    name="b_front_right_linkage">
-    <inertial>
-      <origin
-        xyz="-2.01833246116223E-07 -0.0866174322359831 0.114144894811923"
-        rpy="0 0 0" />
-      <mass
-        value="4.04562727792644" />
-      <inertia
-        ixx="0.140037164042006"
-        ixy="5.57435820882623E-08"
-        ixz="2.08850901566751E-08"
-        iyy="0.0827902917589053"
-        iyz="-0.0400096165626047"
-        izz="0.0604906292211793" />
-    </inertial>
-    <visual>
-      <origin
-        xyz="0 0 0"
-        rpy="0 0 0" />
-      <geometry>
-        <mesh
-          filename="package://trailer_description/meshes/b_front_right_linkage.STL" />
-      </geometry>
-      <material
-        name="">
-        <color
-          rgba="0.792156862745098 0.819607843137255 0.933333333333333 1" />
-      </material>
-    </visual>
-    <collision>
-      <origin
-        xyz="0 0 0"
-        rpy="0 0 0" />
-      <geometry>
-        <mesh
-          filename="package://trailer_description/meshes/b_front_right_linkage.STL" />
-      </geometry>
-    </collision>
-  </link>
-  <joint
-    name="b_front_right_linkage_joint"
+    name="right_linkage">
+    <inertial>
+      <origin
+        xyz="-2.01833246560312E-07 -0.0866174322359837 0.114144894811921"
+        rpy="0 0 0" />
+      <mass
+        value="4.04562727792638" />
+      <inertia
+        ixx="0.140037164042004"
+        ixy="5.5743582091201E-08"
+        ixz="2.08850901407819E-08"
+        iyy="0.0827902917589041"
+        iyz="-0.0400096165626044"
+        izz="0.0604906292211791" />
+    </inertial>
+    <visual>
+      <origin
+        xyz="0 0 0"
+        rpy="0 0 0" />
+      <geometry>
+        <mesh
+          filename="package://trailer_description/meshes/right_linkage.STL" />
+      </geometry>
+      <material
+        name="">
+        <color
+          rgba="0.792156862745098 0.819607843137255 0.933333333333333 1" />
+      </material>
+    </visual>
+    <collision>
+      <origin
+        xyz="0 0 0"
+        rpy="0 0 0" />
+      <geometry>
+        <mesh
+          filename="package://trailer_description/meshes/right_linkage.STL" />
+      </geometry>
+    </collision>
+  </link>
+  <joint
+    name="right_linkage_joint"
     type="revolute">
     <origin
-      xyz="1.46 -0.3625 0"
+      xyz="1.46 -0.385 0"
       rpy="0 0 0" />
     <parent
       link="base_link" />
     <child
-      link="b_front_right_linkage" />
+      link="right_linkage" />
     <axis
       xyz="0 0 1" />
@@ -224,5 +224,5 @@
   </joint>
   <link
-    name="b_front_right_wheel">
+    name="front_right_wheel">
     <inertial>
       <origin
@@ -234,7 +234,7 @@
         ixx="2.08218966287404"
         ixy="1.28145530038214E-18"
-        ixz="-2.40294106238822E-16"
+        ixz="-1.7099551738079E-16"
         iyy="3.08830412900736"
-        iyz="-2.41880721526122E-18"
+        iyz="-2.68534024933067E-18"
         izz="2.08218966287404" />
     </inertial>
@@ -245,24 +245,24 @@
       <geometry>
         <mesh
-          filename="package://trailer_description/meshes/b_front_right_wheel.STL" />
-      </geometry>
-      <material
-        name="">
-        <color
-          rgba="0.792156862745098 0.819607843137255 0.933333333333333 1" />
-      </material>
-    </visual>
-    <collision>
-      <origin
-        xyz="0 0 0"
-        rpy="0 0 0" />
-      <geometry>
-        <mesh
-          filename="package://trailer_description/meshes/b_front_right_wheel.STL" />
-      </geometry>
-    </collision>
-  </link>
-  <joint
-    name="b_front_right_wheel_joint"
+          filename="package://trailer_description/meshes/front_right_wheel.STL" />
+      </geometry>
+      <material
+        name="">
+        <color
+          rgba="0.792156862745098 0.819607843137255 0.933333333333333 1" />
+      </material>
+    </visual>
+    <collision>
+      <origin
+        xyz="0 0 0"
+        rpy="0 0 0" />
+      <geometry>
+        <mesh
+          filename="package://trailer_description/meshes/front_right_wheel.STL" />
+      </geometry>
+    </collision>
+  </link>
+  <joint
+    name="front_right_wheel_joint"
     type="continuous">
     <origin
@@ -270,7 +270,7 @@
       rpy="0 0 0" />
     <parent
-      link="b_front_right_linkage" />
-    <child
-      link="b_front_right_wheel" />
+      link="right_linkage" />
+    <child
+      link="front_right_wheel" />
     <axis
       xyz="0 -1 0" />
@@ -280,5 +280,5 @@
   </joint>
   <link
-    name="b_back_left_wheel">
+    name="rear_left_wheel">
     <inertial>
       <origin
@@ -301,24 +301,24 @@
       <geometry>
         <mesh
-          filename="package://trailer_description/meshes/b_back_left_wheel.STL" />
-      </geometry>
-      <material
-        name="">
-        <color
-          rgba="0.792156862745098 0.819607843137255 0.933333333333333 1" />
-      </material>
-    </visual>
-    <collision>
-      <origin
-        xyz="0 0 0"
-        rpy="0 0 0" />
-      <geometry>
-        <mesh
-          filename="package://trailer_description/meshes/b_back_left_wheel.STL" />
-      </geometry>
-    </collision>
-  </link>
-  <joint
-    name="b_back_left_wheel_joint"
+          filename="package://trailer_description/meshes/rear_left_wheel.STL" />
+      </geometry>
+      <material
+        name="">
+        <color
+          rgba="0.792156862745098 0.819607843137255 0.933333333333333 1" />
+      </material>
+    </visual>
+    <collision>
+      <origin
+        xyz="0 0 0"
+        rpy="0 0 0" />
+      <geometry>
+        <mesh
+          filename="package://trailer_description/meshes/rear_left_wheel.STL" />
+      </geometry>
+    </collision>
+  </link>
+  <joint
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
File: install/trailer_description/share/trailer_description/urdf/trailer_gazebo.xacro (robot description, xacro)
@@ -4,5 +4,5 @@
         <plugin>transmission_interface/SimpleTransmission</plugin>
         <actuator name="left_wheel_motor" role="actuator_left"/>
-        <joint name="b_back_left_wheel_joint" role="joint_left">
+        <joint name="rear_left_wheel_joint" role="joint_left">
             <mechanicalReduction>1.0</mechanicalReduction>
         </joint>
@@ -11,5 +11,5 @@
         <plugin>transmission_interface/SimpleTransmission</plugin>
         <actuator name="right_wheel_motor" role="actuator_right"/>
-        <joint name="b_back_right_wheel_joint" role="joint_right">
+        <joint name="rear_right_wheel_joint" role="joint_right">
             <mechanicalReduction>1.0</mechanicalReduction>
         </joint>
@@ -18,5 +18,5 @@
         <plugin>transmission_interface/SimpleTransmission</plugin>
         <actuator name="left_linkage_actuator" role="actuator_left"/>
-        <joint name="b_front_left_linkage_joint" role="joint_left">
+        <joint name="left_linkage_joint" role="joint_left">
             <mechanicalReduction>1.0</mechanicalReduction>
         </joint>
@@ -25,9 +25,9 @@
         <plugin>transmission_interface/SimpleTransmission</plugin>
         <actuator name="right_linkage_actuator" role="actuator_right"/>
-        <joint name="b_front_right_linkage_joint" role="joint_right">
+        <joint name="right_linkage_joint" role="joint_right">
             <mechanicalReduction>1.0</mechanicalReduction>
         </joint>
     </transmission>
-    <gazebo reference="b_front_left_wheel">
+    <gazebo reference="front_left_wheel">
         <mu1>100000000000000.0</mu1>
         <mu2>100000000000000.0</mu2>
@@ -38,5 +38,5 @@
         <fdir1>0 1 0</fdir1>
     </gazebo>
-    <gazebo reference="b_front_right_wheel">
+    <gazebo reference="front_right_wheel">
         <mu1>100000000000000.0</mu1>
         <mu2>100000000000000.0</mu2>
@@ -47,5 +47,5 @@
         <fdir1>0 -1 0</fdir1>
     </gazebo>
-    <gazebo reference="b_back_left_wheel">
+    <gazebo reference="rear_left_wheel">
         <mu1>100000000000000.0</mu1>
         <mu2>100000000000000.0</mu2>
@@ -56,5 +56,5 @@
         <fdir1>0 1 0</fdir1>
     </gazebo>
-    <gazebo reference="b_fback_right_wheel">
+    <gazebo reference="rear_right_wheel">
         <mu1>100000000000000.0</mu1>
         <mu2>100000000000000.0</mu2>

File: install/trailer_description/share/trailer_description/urdf/trailer_ros2_control.xacro (robot description, xacro)
@@ -6,5 +6,5 @@
         </hardware>
         <!-- Back wheel joints -->
-        <joint name="b_back_left_wheel_joint">
+        <joint name="rear_left_wheel_joint">
             <command_interface name="velocity">
                 <param name="min">-1</param>
@@ -14,5 +14,5 @@
             <state_interface name="velocity"/>
         </joint>
-        <joint name="b_back_right_wheel_joint">
+        <joint name="rear_right_wheel_joint">
             <command_interface name="velocity">
                 <param name="min">-1</param>
@@ -23,5 +23,5 @@
         </joint>
         <!-- Steering linkage joints -->
-        <joint name="b_front_left_linkage_joint">
+        <joint name="left_linkage_joint">
             <command_interface name="position">
                 <param name="min">-0.5</param>
@@ -31,5 +31,5 @@
             <state_interface name="velocity"/>
         </joint>
-        <joint name="b_front_right_linkage_joint">
+        <joint name="right_linkage_joint">
             <command_interface name="position">
                 <param name="min">-0.5</param>
