Commit message: New steering link

File: install/trailer_description/share/trailer_description/urdf/trailer.urdf.xacro (robot description, xacro)
@@ -10,15 +10,15 @@
     <inertial>
       <origin
-        xyz="0.0145343749103901 -4.8067090025433E-11 0.504525903309878"
-        rpy="0 0 0" />
-      <mass
-        value="5621.45261479066" />
-      <inertia
-        ixx="1504.39932306857"
-        ixy="5.67577165358734E-07"
-        ixz="-97.6855056473575"
-        iyy="7926.87309013488"
-        iyz="-6.11751972034413E-08"
-        izz="8441.84332873847" />
+        xyz="0.0151794504413044 -2.72871741278684E-16 0.504333281484515"
+        rpy="0 0 0" />
+      <mass
+        value="5623.96238078164" />
+      <inertia
+        ixx="1505.2735842584"
+        ixy="3.7224720704788E-14"
+        ixz="-96.1203292275202"
+        iyy="7932.64531285603"
+        iyz="-2.22978883011256E-14"
+        izz="8447.43080900142" />
     </inertial>
     <visual>
@@ -52,55 +52,55 @@
   </joint>
   <link
-    name="left_linkage">
-    <inertial>
-      <origin
-        xyz="2.01833246560312E-07 0.086617432235983 0.114144894811922"
-        rpy="0 0 0" />
-      <mass
-        value="4.04562727792638" />
-      <inertia
-        ixx="0.140037164042005"
-        ixy="5.57435821298368E-08"
-        ixz="-2.08850902365895E-08"
-        iyy="0.0827902917589043"
-        iyz="0.0400096165626049"
-        izz="0.0604906292211796" />
-    </inertial>
-    <visual>
-      <origin
-        xyz="0 0 0"
-        rpy="0 0 0" />
-      <geometry>
-        <mesh
-          filename="package://trailer_description/meshes/left_linkage.STL" />
-      </geometry>
-      <material
-        name="">
-        <color
-          rgba="0.792156862745098 0.819607843137255 0.933333333333333 1" />
-      </material>
-    </visual>
-    <collision>
-      <origin
-        xyz="0 0 0"
-        rpy="0 0 0" />
-      <geometry>
-        <mesh
-          filename="package://trailer_description/meshes/left_linkage.STL" />
-      </geometry>
-    </collision>
-  </link>
-  <joint
-    name="left_linkage_joint"
+    name="steer_left">
+    <inertial>
+      <origin
+        xyz="0 0 1.11022302462516E-16"
+        rpy="0 0 0" />
+      <mass
+        value="1.48283173249438" />
+      <inertia
+        ixx="0.0113467519863581"
+        ixy="4.92526541296846E-36"
+        ixz="0"
+        iyy="0.00118626538599551"
+        iyz="4.00998451212503E-35"
+        izz="0.0113467519863581" />
+    </inertial>
+    <visual>
+      <origin
+        xyz="0 0 0"
+        rpy="0 0 0" />
+      <geometry>
+        <mesh
+          filename="package://trailer_description/meshes/steer_left.STL" />
+      </geometry>
+      <material
+        name="">
+        <color
+          rgba="0.792156862745098 0.819607843137255 0.933333333333333 1" />
+      </material>
+    </visual>
+    <collision>
+      <origin
+        xyz="0 0 0"
+        rpy="0 0 0" />
+      <geometry>
+        <mesh
+          filename="package://trailer_description/meshes/steer_left.STL" />
+      </geometry>
+    </collision>
+  </link>
+  <joint
+    name="steer_left_joint"
     type="revolute">
     <origin
-      xyz="1.46 0.385 0"
+      xyz="1.46 0.6125 0"
       rpy="0 0 0" />
     <parent
       link="base_link" />
     <child
-      link="left_linkage" />
-    <axis
-      xyz="0 0 1" />
+      link="steer_left" />
+    <axis
+      xyz="0 0 -1" />
     <limit
       lower="-0.5"
@@ -113,5 +113,5 @@
     <inertial>
       <origin
-        xyz="0 0 0"
+        xyz="0 0 -1.11022302462516E-16"
         rpy="0 0 0" />
       <mass
@@ -119,8 +119,8 @@
       <inertia
         ixx="2.08218966287404"
-        ixy="-1.30089087994337E-17"
-        ixz="5.1605164674113E-17"
+        ixy="6.07695317678125E-17"
+        ixz="-3.14934790723029E-18"
         iyy="3.08830412900736"
-        iyz="7.48293486257905E-18"
+        iyz="3.93136225252298E-18"
         izz="2.08218966287404" />
     </inertial>
@@ -153,66 +153,66 @@
     type="continuous">
     <origin
-      xyz="0 0.2275 0"
-      rpy="0 0 0" />
-    <parent
-      link="left_linkage" />
+      xyz="0 0 0"
+      rpy="0 0 0" />
+    <parent
+      link="steer_left" />
     <child
       link="front_left_wheel" />
     <axis
-      xyz="0 -1 0" />
-    <limit
+      xyz="0 1 0" />
+      <limit
       effort="100"
       velocity="31.4" />
   </joint>
   <link
-    name="right_linkage">
-    <inertial>
-      <origin
-        xyz="-2.01833246560312E-07 -0.0866174322359837 0.114144894811921"
-        rpy="0 0 0" />
-      <mass
-        value="4.04562727792638" />
-      <inertia
-        ixx="0.140037164042004"
-        ixy="5.5743582091201E-08"
-        ixz="2.08850901407819E-08"
-        iyy="0.0827902917589041"
-        iyz="-0.0400096165626044"
-        izz="0.0604906292211791" />
-    </inertial>
-    <visual>
-      <origin
-        xyz="0 0 0"
-        rpy="0 0 0" />
-      <geometry>
-        <mesh
-          filename="package://trailer_description/meshes/right_linkage.STL" />
-      </geometry>
-      <material
-        name="">
-        <color
-          rgba="0.792156862745098 0.819607843137255 0.933333333333333 1" />
-      </material>
-    </visual>
-    <collision>
-      <origin
-        xyz="0 0 0"
-        rpy="0 0 0" />
-      <geometry>
-        <mesh
-          filename="package://trailer_description/meshes/right_linkage.STL" />
-      </geometry>
-    </collision>
-  </link>
-  <joint
-    name="right_linkage_joint"
+    name="steer_right">
+    <inertial>
+      <origin
+        xyz="0 0 1.11022302462516E-16"
+        rpy="0 0 0" />
+      <mass
+        value="1.48283173249438" />
+      <inertia
+        ixx="0.0113467519863581"
+        ixy="4.92526541296846E-36"
+        ixz="0"
+        iyy="0.00118626538599551"
+        iyz="4.00998451212503E-35"
+        izz="0.0113467519863581" />
+    </inertial>
+    <visual>
+      <origin
+        xyz="0 0 0"
+        rpy="0 0 0" />
+      <geometry>
+        <mesh
+          filename="package://trailer_description/meshes/steer_right.STL" />
+      </geometry>
+      <material
+        name="">
+        <color
+          rgba="0.792156862745098 0.819607843137255 0.933333333333333 1" />
+      </material>
+    </visual>
+    <collision>
+      <origin
+        xyz="0 0 0"
+        rpy="0 0 0" />
+      <geometry>
+        <mesh
+          filename="package://trailer_description/meshes/steer_right.STL" />
+      </geometry>
+    </collision>
+  </link>
+  <joint
+    name="steer_right_joint"
     type="revolute">
     <origin
-      xyz="1.46 -0.385 0"
+      xyz="1.46 -0.6125 0"
       rpy="0 0 0" />
     <parent
       link="base_link" />
     <child
-      link="right_linkage" />
+      link="steer_right" />
     <axis
       xyz="0 0 1" />
@@ -227,5 +227,5 @@
     <inertial>
       <origin
-        xyz="0 0 0"
+        xyz="0 0 -1.11022302462516E-16"
         rpy="0 0 0" />
       <mass
@@ -233,8 +233,8 @@
       <inertia
         ixx="2.08218966287404"
-        ixy="1.28145530038214E-18"
-        ixz="-1.7099551738079E-16"
+        ixy="6.07695317678125E-17"
+        ixz="1.71424910145489E-17"
         iyy="3.08830412900736"
-        iyz="-2.68534024933067E-18"
+        iyz="1.83241460922682E-18"
         izz="2.08218966287404" />
     </inertial>
@@ -267,13 +267,13 @@
     type="continuous">
     <origin
-      xyz="0 -0.2275 0"
-      rpy="0 0 0" />
-    <parent
-      link="right_linkage" />
+      xyz="0 0 0"
+      rpy="0 0 0" />
+    <parent
+      link="steer_right" />
     <child
       link="front_right_wheel" />
     <axis
-      xyz="0 -1 0" />
-    <limit
+      xyz="0 1 0" />
+      <limit
       effort="100"
       velocity="31.4" />
@@ -395,5 +395,5 @@
     <inertial>
       <origin
-        xyz="-2.06473943000056 -9.13851883438585E-17 0.256889099220807"
+        xyz="-2.06473943000056 -9.59060549514745E-17 0.256889099220807"
         rpy="0 0 0" />
       <mass
@@ -401,8 +401,8 @@
       <inertia
         ixx="634.919956534306"
-        ixy="7.69341401721132E-14"
-        ixz="9.2945345694552"
+        ixy="7.66014195843368E-14"
+        ixz="9.29453456945521"
         iyy="1640.30654615615"
-        iyz="5.72407813967429E-15"
+        iyz="4.53164968888437E-15"
         izz="2004.11171155846" />
     </inertial>

File: install/trailer_description/share/trailer_description/urdf/trailer_gazebo.xacro (robot description, xacro)
@@ -15,15 +15,15 @@
         </joint>
     </transmission>
-    <transmission name="left_linkage_transmission">
+    <transmission name="left_steer_transmission">
         <plugin>transmission_interface/SimpleTransmission</plugin>
-        <actuator name="left_linkage_actuator" role="actuator_left"/>
-        <joint name="left_linkage_joint" role="joint_left">
+        <actuator name="left_steer_actuator" role="actuator_left"/>
+        <joint name="steer_left_joint" role="joint_left">
             <mechanicalReduction>1.0</mechanicalReduction>
         </joint>
     </transmission>
-    <transmission name="right_linkage_transmission">
+    <transmission name="right_steer_transmission">
         <plugin>transmission_interface/SimpleTransmission</plugin>
-        <actuator name="right_linkage_actuator" role="actuator_right"/>
-        <joint name="right_linkage_joint" role="joint_right">
+        <actuator name="right_steer_actuator" role="actuator_right"/>
+        <joint name="steer_right_joint" role="joint_right">
             <mechanicalReduction>1.0</mechanicalReduction>
         </joint>

File: install/trailer_description/share/trailer_description/urdf/trailer_ros2_control.xacro (robot description, xacro)
@@ -23,5 +23,5 @@
         </joint>
         <!-- Steering linkage joints -->
-        <joint name="left_linkage_joint">
+        <joint name="steer_left_joint">
             <command_interface name="position">
                 <param name="min">-0.5</param>
@@ -31,5 +31,5 @@
             <state_interface name="velocity"/>
         </joint>
-        <joint name="right_linkage_joint">
+        <joint name="steer_right_joint">
             <command_interface name="position">
                 <param name="min">-0.5</param>

File: src/trailer_description/urdf/trailer.urdf copy.xacro (robot description, xacro)
@@ -10,15 +10,15 @@
     <inertial>
       <origin
-        xyz="0.0151794504413044 -2.72871741278684E-16 0.504333281484515"
-        rpy="0 0 0" />
-      <mass
-        value="5623.96238078164" />
-      <inertia
-        ixx="1505.2735842584"
-        ixy="3.7224720704788E-14"
-        ixz="-96.1203292275202"
-        iyy="7932.64531285603"
-        iyz="-2.22978883011256E-14"
-        izz="8447.43080900142" />
+        xyz="0.0145343749103901 -4.8067090025433E-11 0.504525903309878"
+        rpy="0 0 0" />
+      <mass
+        value="5621.45261479066" />
+      <inertia
+        ixx="1504.39932306857"
+        ixy="5.67577165358734E-07"
+        ixz="-97.6855056473575"
+        iyy="7926.87309013488"
+        iyz="-6.11751972034413E-08"
+        izz="8441.84332873847" />
     </inertial>
     <visual>
@@ -52,55 +52,55 @@
   </joint>
   <link
-    name="steer_left">
-    <inertial>
-      <origin
-        xyz="0 0 1.11022302462516E-16"
-        rpy="0 0 0" />
-      <mass
-        value="1.48283173249438" />
-      <inertia
-        ixx="0.0113467519863581"
-        ixy="4.92526541296846E-36"
-        ixz="0"
-        iyy="0.00118626538599551"
-        iyz="4.00998451212503E-35"
-        izz="0.0113467519863581" />
-    </inertial>
-    <visual>
-      <origin
-        xyz="0 0 0"
-        rpy="0 0 0" />
-      <geometry>
-        <mesh
-          filename="package://trailer_description/meshes/steer_left.STL" />
-      </geometry>
-      <material
-        name="">
-        <color
-          rgba="0.792156862745098 0.819607843137255 0.933333333333333 1" />
-      </material>
-    </visual>
-    <collision>
-      <origin
-        xyz="0 0 0"
-        rpy="0 0 0" />
-      <geometry>
-        <mesh
-          filename="package://trailer_description/meshes/steer_left.STL" />
-      </geometry>
-    </collision>
-  </link>
-  <joint
-    name="steer_left_joint"
+    name="left_linkage">
+    <inertial>
+      <origin
+        xyz="2.01833246560312E-07 0.086617432235983 0.114144894811922"
+        rpy="0 0 0" />
+      <mass
+        value="4.04562727792638" />
+      <inertia
+        ixx="0.140037164042005"
+        ixy="5.57435821298368E-08"
+        ixz="-2.08850902365895E-08"
+        iyy="0.0827902917589043"
+        iyz="0.0400096165626049"
+        izz="0.0604906292211796" />
+    </inertial>
+    <visual>
+      <origin
+        xyz="0 0 0"
+        rpy="0 0 0" />
+      <geometry>
+        <mesh
+          filename="package://trailer_description/meshes/left_linkage.STL" />
+      </geometry>
+      <material
+        name="">
+        <color
+          rgba="0.792156862745098 0.819607843137255 0.933333333333333 1" />
+      </material>
+    </visual>
+    <collision>
+      <origin
+        xyz="0 0 0"
+        rpy="0 0 0" />
+      <geometry>
+        <mesh
+          filename="package://trailer_description/meshes/left_linkage.STL" />
+      </geometry>
+    </collision>
+  </link>
+  <joint
+    name="left_linkage_joint"
     type="revolute">
     <origin
-      xyz="1.46 0.6125 0"
+      xyz="1.46 0.385 0"
       rpy="0 0 0" />
     <parent
       link="base_link" />
     <child
-      link="steer_left" />
-    <axis
-      xyz="0 0 -1" />
+      link="left_linkage" />
+    <axis
+      xyz="0 0 1" />
     <limit
       lower="-0.5"
@@ -113,5 +113,5 @@
     <inertial>
       <origin
-        xyz="0 0 -1.11022302462516E-16"
+        xyz="0 0 0"
         rpy="0 0 0" />
       <mass
@@ -119,8 +119,8 @@
       <inertia
         ixx="2.08218966287404"
-        ixy="6.07695317678125E-17"
-        ixz="-3.14934790723029E-18"
+        ixy="-1.30089087994337E-17"
+        ixz="5.1605164674113E-17"
         iyy="3.08830412900736"
-        iyz="3.93136225252298E-18"
+        iyz="7.48293486257905E-18"
         izz="2.08218966287404" />
     </inertial>
@@ -153,66 +153,66 @@
     type="continuous">
     <origin
-      xyz="0 0 0"
-      rpy="0 0 0" />
-    <parent
-      link="steer_left" />
+      xyz="0 0.2275 0"
+      rpy="0 0 0" />
+    <parent
+      link="left_linkage" />
     <child
       link="front_left_wheel" />
     <axis
-      xyz="0 1 0" />
-      <limit
+      xyz="0 -1 0" />
+    <limit
       effort="100"
       velocity="31.4" />
   </joint>
   <link
-    name="steer_right">
-    <inertial>
-      <origin
-        xyz="0 0 1.11022302462516E-16"
-        rpy="0 0 0" />
-      <mass
-        value="1.48283173249438" />
-      <inertia
-        ixx="0.0113467519863581"
-        ixy="4.92526541296846E-36"
-        ixz="0"
-        iyy="0.00118626538599551"
-        iyz="4.00998451212503E-35"
-        izz="0.0113467519863581" />
-    </inertial>
-    <visual>
-      <origin
-        xyz="0 0 0"
-        rpy="0 0 0" />
-      <geometry>
-        <mesh
-          filename="package://trailer_description/meshes/steer_right.STL" />
-      </geometry>
-      <material
-        name="">
-        <color
-          rgba="0.792156862745098 0.819607843137255 0.933333333333333 1" />
-      </material>
-    </visual>
-    <collision>
-      <origin
-        xyz="0 0 0"
-        rpy="0 0 0" />
-      <geometry>
-        <mesh
-          filename="package://trailer_description/meshes/steer_right.STL" />
-      </geometry>
-    </collision>
-  </link>
-  <joint
-    name="steer_right_joint"
+    name="right_linkage">
+    <inertial>
+      <origin
+        xyz="-2.01833246560312E-07 -0.0866174322359837 0.114144894811921"
+        rpy="0 0 0" />
+      <mass
+        value="4.04562727792638" />
+      <inertia
+        ixx="0.140037164042004"
+        ixy="5.5743582091201E-08"
+        ixz="2.08850901407819E-08"
+        iyy="0.0827902917589041"
+        iyz="-0.0400096165626044"
+        izz="0.0604906292211791" />
+    </inertial>
+    <visual>
+      <origin
+        xyz="0 0 0"
+        rpy="0 0 0" />
+      <geometry>
+        <mesh
+          filename="package://trailer_description/meshes/right_linkage.STL" />
+      </geometry>
+      <material
+        name="">
+        <color
+          rgba="0.792156862745098 0.819607843137255 0.933333333333333 1" />
+      </material>
+    </visual>
+    <collision>
+      <origin
+        xyz="0 0 0"
+        rpy="0 0 0" />
+      <geometry>
+        <mesh
+          filename="package://trailer_description/meshes/right_linkage.STL" />
+      </geometry>
+    </collision>
+  </link>
+  <joint
+    name="right_linkage_joint"
     type="revolute">
     <origin
-      xyz="1.46 -0.6125 0"
+      xyz="1.46 -0.385 0"
       rpy="0 0 0" />
     <parent
       link="base_link" />
     <child
-      link="steer_right" />
+      link="right_linkage" />
     <axis
       xyz="0 0 1" />
@@ -227,5 +227,5 @@
     <inertial>
       <origin
-        xyz="0 0 -1.11022302462516E-16"
+        xyz="0 0 0"
         rpy="0 0 0" />
       <mass
@@ -233,8 +233,8 @@
       <inertia
         ixx="2.08218966287404"
-        ixy="6.07695317678125E-17"
-        ixz="1.71424910145489E-17"
+        ixy="1.28145530038214E-18"
+        ixz="-1.7099551738079E-16"
         iyy="3.08830412900736"
-        iyz="1.83241460922682E-18"
+        iyz="-2.68534024933067E-18"
         izz="2.08218966287404" />
     </inertial>
@@ -267,13 +267,13 @@
     type="continuous">
     <origin
-      xyz="0 0 0"
-      rpy="0 0 0" />
-    <parent
-      link="steer_right" />
+      xyz="0 -0.2275 0"
+      rpy="0 0 0" />
+    <parent
+      link="right_linkage" />
     <child
       link="front_right_wheel" />
     <axis
-      xyz="0 1 0" />
-      <limit
+      xyz="0 -1 0" />
+    <limit
       effort="100"
       velocity="31.4" />
@@ -395,5 +395,5 @@
     <inertial>
       <origin
-        xyz="-2.06473943000056 -9.59060549514745E-17 0.256889099220807"
+        xyz="-2.06473943000056 -9.13851883438585E-17 0.256889099220807"
         rpy="0 0 0" />
       <mass
@@ -401,8 +401,8 @@
       <inertia
         ixx="634.919956534306"
-        ixy="7.66014195843368E-14"
-        ixz="9.29453456945521"
+        ixy="7.69341401721132E-14"
+        ixz="9.2945345694552"
         iyy="1640.30654615615"
-        iyz="4.53164968888437E-15"
+        iyz="5.72407813967429E-15"
         izz="2004.11171155846" />
     </inertial>

File: src/trailer_description/urdf/trailer_assembly.urdf (robot description, URDF)
Before this commit: robot trailer, 11 links, 10 joints
Links:
- removed link base_footprint
- link base_link: geometry collision mesh filename=package://trailer_assembly/meshes/base_link.STL; visual mesh filename=package://trailer_assembly/meshes/base_link.STL
- link front_left_wheel: geometry collision mesh filename=package://trailer_assembly/meshes/front_left_wheel.STL; visual mesh filename=package://trailer_assembly/meshes/front_left_wheel.STL
- link front_right_wheel: geometry collision mesh filename=package://trailer_assembly/meshes/front_right_wheel.STL; visual mesh filename=package://trailer_assembly/meshes/front_right_wheel.STL
- link rear_left_wheel: geometry collision mesh filename=package://trailer_assembly/meshes/rear_left_wheel.STL; visual mesh filename=package://trailer_assembly/meshes/rear_left_wheel.STL
- link rear_right_wheel: geometry collision mesh filename=package://trailer_assembly/meshes/rear_right_wheel.STL; visual mesh filename=package://trailer_assembly/meshes/rear_right_wheel.STL
- link steer_left: geometry collision mesh filename=package://trailer_assembly/meshes/steer_left.STL; visual mesh filename=package://trailer_assembly/meshes/steer_left.STL
- link steer_right: geometry collision mesh filename=package://trailer_assembly/meshes/steer_right.STL; visual mesh filename=package://trailer_assembly/meshes/steer_right.STL
- link t_left_wheel: geometry collision mesh filename=package://trailer_assembly/meshes/t_left_wheel.STL; visual mesh filename=package://trailer_assembly/meshes/t_left_wheel.STL
- link t_right_wheel: geometry collision mesh filename=package://trailer_assembly/meshes/t_right_wheel.STL; visual mesh filename=package://trailer_assembly/meshes/t_right_wheel.STL
- link trailer: geometry collision mesh filename=package://trailer_assembly/meshes/trailer.STL; visual mesh filename=package://trailer_assembly/meshes/trailer.STL
Joints:
- removed joint base_joint
- joint front_left_wheel_joint: limit effort=100 velocity=31.4 -> (none)
- joint front_right_wheel_joint: limit effort=100 velocity=31.4 -> (none)
- joint rear_left_wheel_joint: limit effort=100 velocity=31.4 -> lower=0 upper=0 effort=100 velocity=31.4
- joint rear_right_wheel_joint: limit effort=100 velocity=31.4 -> lower=0 upper=0 effort=100 velocity=31.4
- joint steer_left_joint: limit lower=-0.5 upper=0.5 effort=50 velocity=1.5 -> lower=0 upper=0 effort=100 velocity=31.4
- joint steer_right_joint: limit lower=-0.5 upper=0.5 effort=50 velocity=1.5 -> lower=0 upper=0 effort=100 velocity=31.4
- joint t_left_wheel_joint: limit effort=100 velocity=31.4 -> lower=0 upper=0 effort=100 velocity=31.4
- joint t_right_wheel_joint: limit effort=100 velocity=31.4 -> lower=0 upper=0 effort=100 velocity=31.4
