Commit message: Added imu to the xacro and gazebo file

File: install/trailer_description/share/trailer_description/urdf/trailer.urdf.xacro (robot description, xacro)
@@ -561,3 +561,31 @@
       velocity="31.4" />
   </joint>
+  <link name="imu_link">
+    <inertial>
+      <mass value="0.01"/>
+      <origin xyz="0.0 0 0" rpy="0 0 0"/>
+      <inertia
+          ixx="1e-7" ixy="0" ixz="0"
+          iyy="1e-7" iyz="0"
+          izz="1e-7"
+      />
+  </inertial>
+    <visual>
+      <origin xyz="0 0 0" rpy="0 0 0"/>
+      <geometry>
+        <box size="0.001 0.001 0.001"/>
+      </geometry>
+    </visual>
+    <collision>
+      <origin xyz="0 0 0" rpy="0 0 0"/>
+      <geometry>
+        <box size="0.001 0.001 0.001"/>
+      </geometry>
+    </collision>
+  </link>
+  <joint name="imu_joint" type="fixed">
+    <origin xyz="0 0 0" rpy="0 0 0"/>
+    <parent link="base_link"/>
+    <child link="imu_link"/>
+  </joint>
 </robot>

File: install/trailer_description/share/trailer_description/urdf/trailer_gazebo.xacro (robot description, xacro)
@@ -117,3 +117,52 @@
         </plugin>
     </gazebo>
+    <gazebo reference="imu_link">
+        <sensor type="imu" name="imu">
+            <always_on>true</always_on>
+            <update_rate>100</update_rate>
+            <imu>
+                <angular_velocity>
+                    <x>
+                        <noise type="gaussian">
+                            <mean>0.0</mean>
+                            <stddev>2e-4</stddev>
+                        </noise>
+                    </x>
+                    <y>
+                        <noise type="gaussian">
+                            <mean>0.0</mean>
+                            <stddev>2e-4</stddev>
+                        </noise>
+                    </y>
+                    <z>
+                        <noise type="gaussian">
+                            <mean>0.0</mean>
+                            <stddev>2e-4</stddev>
+                        </noise>
+                    </z>
+                </angular_velocity>
+                <linear_acceleration>
+                    <x>
+                        <noise type="gaussian">
+                            <mean>0.0</mean>
+                            <stddev>1.7e-2</stddev>
+                        </noise>
+                    </x>
+                    <y>
+                        <noise type="gaussian">
+                            <mean>0.0</mean>
+                            <stddev>1.7e-2</stddev>
+                        </noise>
+                    </y>
+                    <z>
+                        <noise type="gaussian">
+                            <mean>0.0</mean>
+                            <stddev>1.7e-2</stddev>
+                        </noise>
+                    </z>
+                </linear_acceleration>
+            </imu>
+            <plugin filename="libgazebo_ros_imu_sensor.so" name="imu"/>
+        </sensor>
+    </gazebo>
 </robot>

Commit message: Added 4 ultrasonic sensors and one depth camera. But the position is incorrect and the topics are not published

File: install/trailer_description/share/trailer_description/urdf/trailer.urdf.xacro (robot description, xacro)
@@ -589,3 +589,55 @@
     <child link="imu_link"/>
   </joint>
+<!-- Ultrasonic Sensors -->
+<xacro:macro name="ultrasonic_sensor" params="name x y z">
+  <link name="${name}">
+    <visual>
+      <origin xyz="${x} ${y} ${z}" rpy="0 0 0"/>
+      <geometry>
+        <cylinder length="0.02" radius="0.015"/>
+      </geometry>
+      <material name="sensor_mat">
+        <color rgba="0.5 0.5 0.5 1"/>
+      </material>
+    </visual>
+  </link>
+  <joint name="${name}_joint" type="fixed">
+    <origin xyz="${x} ${y} ${z}" rpy="0 0 0"/>
+    <parent link="base_link"/>
+    <child link="${name}"/>
+  </joint>
+</xacro:macro>
+<!-- Add Ultrasonic Sensors -->
+<xacro:ultrasonic_sensor name="u1_link" x="-2.16" y="0.6125" z="0.05"/>
+<xacro:ultrasonic_sensor name="u2_link" x="-2.16" y="0.26" z="0.05"/>
+<xacro:ultrasonic_sensor name="u3_link" x="-2.16" y="-0.26" z="0.05"/>
+<xacro:ultrasonic_sensor name="u4_link" x="-2.16" y="-0.6125" z="0.05"/>
+<!-- Depth Sense Camera -->
+<link name="depth_camera_link">
+  <inertial>
+    <origin xyz="0 0 0" rpy="0 0 0"/>
+    <mass value="0.1"/>
+    <inertia ixx="1e-6" ixy="0" ixz="0" iyy="1e-6" iyz="0" izz="1e-6"/>
+  </inertial>
+  <visual>
+    <origin xyz="-2.16 0 0.41495" rpy="0 0 0"/>
+    <geometry>
+      <box size="0.02 0.06 0.015"/>
+    </geometry>
+    <material name="depth_camera_material">
+      <color rgba="0.5 0.5 0.5 1.0"/>
+    </material>
+  </visual>
+  <collision>
+    <origin xyz="-2.16 0 0.41495" rpy="0 0 0"/>
+    <geometry>
+      <box size="0.02 0.06 0.015"/>
+    </geometry>
+  </collision>
+</link>
+<joint name="depth_camera_joint" type="fixed">
+  <origin xyz="-2.16 0 0.41495" rpy="0 0 0"/>
+  <parent link="base_link"/>
+  <child link="depth_camera_link"/>
+</joint>
 </robot>

File: install/trailer_description/share/trailer_description/urdf/trailer_gazebo.xacro (robot description, xacro)
@@ -166,3 +166,162 @@
         </sensor>
     </gazebo>
+    <!-- Ultrasonic Sensor u1 -->
+    <gazebo reference="u1_link">
+        <sensor type="ray" name="ultrasonic_sensor_u1">
+            <pose>-2.16 0.6125 0.05 0 0 0</pose>
+            <visualize>true</visualize>
+            <update_rate>10</update_rate>
+            <ray>
+                <scan>
+                    <horizontal>
+                        <samples>1</samples>
+                        <resolution>1</resolution>
+                        <min_angle>0</min_angle>
+                        <max_angle>0</max_angle>
+                    </horizontal>
+                </scan>
+                <range>
+                    <min>0.02</min>
+                    <max>4.0</max>
+                    <resolution>0.01</resolution>
+                </range>
+            </ray>
+            <plugin filename="libgazebo_ros_range.so" name="gazebo_ros_ultrasonic_u1">
+                <gaussianNoise>0.01</gaussianNoise>
+                <alwaysOn>true</alwaysOn>
+                <updateRate>10</updateRate>
+                <topicName>sensor/ultrasonic_u1</topicName>
+                <frameName>u1_link</frameName>
+                <radiation>ultrasonic</radiation>
+            </plugin>
+        </sensor>
+    </gazebo>
+    <!-- Ultrasonic Sensor u2 -->
+    <gazebo reference="u2_link">
+        <sensor type="ray" name="ultrasonic_sensor_u2">
+            <pose>-2.16 0.260 0.05 0 0 0</pose>
+            <visualize>true</visualize>
+            <update_rate>10</update_rate>
+            <ray>
+                <scan>
+                    <horizontal>
+                        <samples>1</samples>
+                        <resolution>1</resolution>
+                        <min_angle>0</min_angle>
+                        <max_angle>0</max_angle>
+                    </horizontal>
+                </scan>
+                <range>
+                    <min>0.02</min>
+                    <max>4.0</max>
+                    <resolution>0.01</resolution>
+                </range>
+            </ray>
+            <plugin filename="libgazebo_ros_range.so" name="gazebo_ros_ultrasonic_u2">
+                <gaussianNoise>0.01</gaussianNoise>
+                <alwaysOn>true</alwaysOn>
+                <updateRate>10</updateRate>
+                <topicName>sensor/ultrasonic_u2</topicName>
+                <frameName>u2_link</frameName>
+                <radiation>ultrasonic</radiation>
+            </plugin>
+        </sensor>
+    </gazebo>
+    <!-- Ultrasonic Sensor u3 -->
+    <gazebo reference="u3_link">
+        <sensor type="ray" name="ultrasonic_sensor_u3">
+            <pose>-2.16 -0.260 0.05 0 0 0</pose>
+            <visualize>true</visualize>
+            <update_rate>10</update_rate>
+            <ray>
+                <scan>
+                    <horizontal>
+                        <samples>1</samples>
+                        <resolution>1</resolution>
+                        <min_angle>0</min_angle>
+                        <max_angle>0</max_angle>
+                    </horizontal>
+                </scan>
+                <range>
+                    <min>0.02</min>
+                    <max>4.0</max>
+                    <resolution>0.01</resolution>
+                </range>
+            </ray>
+            <plugin filename="libgazebo_ros_range.so" name="gazebo_ros_ultrasonic_u3">
+                <gaussianNoise>0.01</gaussianNoise>
+                <alwaysOn>true</alwaysOn>
+                <updateRate>10</updateRate>
+                <topicName>sensor/ultrasonic_u3</topicName>
+                <frameName>u3_link</frameName>
+                <radiation>ultrasonic</radiation>
+            </plugin>
+        </sensor>
+    </gazebo>
+    <!-- Ultrasonic Sensor u4 -->
+    <gazebo reference="u4_link">
+        <sensor type="ray" name="ultrasonic_sensor_u4">
+            <pose>-2.16 -0.6125 0.05 0 0 0</pose>
+            <visualize>true</visualize>
+            <update_rate>10</update_rate>
+            <ray>
+                <scan>
+                    <horizontal>
+                        <samples>1</samples>
+                        <resolution>1</resolution>
+                        <min_angle>0</min_angle>
+                        <max_angle>0</max_angle>
+                    </horizontal>
+                </scan>
+                <range>
+                    <min>0.02</min>
+                    <max>4.0</max>
+                    <resolution>0.01</resolution>
+                </range>
+            </ray>
+            <plugin filename="libgazebo_ros_range.so" name="gazebo_ros_ultrasonic_u4">
+                <gaussianNoise>0.01</gaussianNoise>
+                <alwaysOn>true</alwaysOn>
+                <updateRate>10</updateRate>
+                <topicName>sensor/ultrasonic_u4</topicName>
+                <frameName>u4_link</frameName>
+                <radiation>ultrasonic</radiation>
+            </plugin>
+        </sensor>
+    </gazebo>
+    <!-- Depth Camera Setup -->
+    <gazebo reference="depth_camera_link">
+        <sensor name="depth_camera" type="depth">
+            <pose>0.0 0.0 0.0 0.0 0.0 0.0</pose>
+            <always_on>true</always_on>
+            <visualize>true</visualize>
+            <update_rate>30.0</update_rate>
+            <camera name="depth_camera">
+            <horizontal_fov>1.23918</horizontal_fov>
+            <image>
+                <width>640</width>
+                <height>480</height>
+                <format>R8G8B8</format>
+            </image>
+            <clip>
+                <near>0.02</near>
+                <far>300</far>
+            </clip>
+            </camera>
+            <plugin name="gazebo_ros_depth_camera_plugin" filename="libgazebo_ros_openni_kinect.so">
+                <baseline>0.2</baseline>
+                <alwaysOn>true</alwaysOn>
+                <updateRate>0.0</updateRate>
+                <cameraName>depth_camera</cameraName>
+                <imageTopicName>/trailer/color/image_raw</imageTopicName>
+                <cameraInfoTopicName>/trailer/color/camera_info</cameraInfoTopicName>
+                <depthImageTopicName>/trailer/depth/image_raw</depthImageTopicName>
+                <depthImageCameraInfoTopicName>/trailer/depth/camera_info</depthImageCameraInfoTopicName>
+                <pointCloudTopicName>/trailer/depth/points</pointCloudTopicName>
+                <frameName>depth_camera_link</frameName>
+                <pointCloudCutoff>0.5</pointCloudCutoff>
+                <pointCloudCutoffMax>3.0</pointCloudCutoffMax>
+            </plugin>
+        </sensor>
+    </gazebo>
 </robot>
