Commit message: .

File: install/trailer_description/share/trailer_description/urdf/trailer.urdf.xacro (robot description, xacro)
@@ -5,4 +5,5 @@
   <xacro:include filename="$(find trailer_description)/urdf/trailer_gazebo.xacro"/>
   <xacro:include filename="$(find trailer_description)/urdf/trailer_ros2_control.xacro"/>
+  <xacro:include filename="$(find trailer_description)/urdf/trailer_material.xacro"/>
   <link name="base_footprint"/>
   <link
@@ -10,5 +11,5 @@
     <inertial>
       <origin
-        xyz="0.0151794504413042 -2.70446273320019E-16 0.504333281484515"
+        xyz="0.0151794504413043 -2.70548710772098E-16 0.504333281484515"
         rpy="0 0 0" />
       <mass
@@ -16,8 +17,8 @@
       <inertia
         ixx="1505.2735842584"
-        ixy="2.45552732709707E-14"
+        ixy="2.80968637770799E-14"
         ixz="-96.1203292275202"
-        iyy="7932.64531285603"
-        iyz="-2.74532801802233E-14"
+        iyy="7932.64531285604"
+        iyz="-2.5937462802081E-14"
         izz="8447.43080900142" />
     </inertial>
@@ -395,5 +396,5 @@
     <inertial>
       <origin
-        xyz="-2.06473943000056 -9.65449692159716E-17 0.256889099220807"
+        xyz="-2.06473943000056 -9.58261906684124E-17 0.256889099220807"
         rpy="0 0 0" />
       <mass
@@ -401,8 +402,8 @@
       <inertia
         ixx="634.919956534306"
-        ixy="7.7271657034793E-14"
-        ixz="9.29453456945518"
+        ixy="7.70909607408193E-14"
+        ixz="9.2945345694552"
         iyy="1640.30654615615"
-        iyz="4.81260634396325E-15"
+        iyz="5.74506370494421E-15"
         izz="2004.11171155846" />
     </inertial>
@@ -453,5 +454,5 @@
     <inertial>
       <origin
-        xyz="0 0 1.11022302462516E-16"
+        xyz="0 0 0"
         rpy="0 0 0" />
       <mass
@@ -515,5 +516,5 @@
       <inertia
         ixx="2.08218966287404"
-        ixy="-1.11352546000203E-18"
+        ixy="-1.11352546000202E-18"
         ixz="6.83908165898515E-17"
         iyy="3.08830412900736"
@@ -595,5 +596,5 @@
     <inertial>
       <origin
-        xyz="-2.22044604925031E-16 0 0"
+        xyz="2.22044604925031E-16 0 0"
         rpy="0 0 0" />
       <mass
@@ -602,7 +603,7 @@
         ixx="4.97009775274937E-08"
         ixy="6.44944990373328E-23"
-        ixz="1.28060738442034E-40"
+        ixz="-1.28060738442034E-40"
         iyy="3.95767043274481E-08"
-        iyz="-9.95682444457783E-55"
+        iyz="9.95682444457783E-55"
         izz="3.95767043274481E-08" />
     </inertial>
@@ -636,5 +637,5 @@
     <origin
       xyz="-2.16 0.6125 0.05"
-      rpy="0 0 0" />
+      rpy="0 0 3.1416" />
     <parent
       link="base_link" />
@@ -648,5 +649,5 @@
     <inertial>
       <origin
-        xyz="-4.44089209850063E-16 0 0"
+        xyz="4.44089209850063E-16 0 0"
         rpy="0 0 0" />
       <mass
@@ -655,7 +656,7 @@
         ixx="4.97009775274937E-08"
         ixy="-6.61984950467753E-23"
-        ixz="-6.44944990373324E-23"
+        ixz="6.44944990373324E-23"
         iyy="3.95767043274481E-08"
-        iyz="1.03497225198971E-37"
+        iyz="-1.03497225198971E-37"
         izz="3.95767043274481E-08" />
     </inertial>
@@ -689,5 +690,5 @@
     <origin
       xyz="-2.16 0.26 0.05"
-      rpy="0 0 0" />
+      rpy="0 0 3.1416" />
     <parent
       link="base_link" />
@@ -701,5 +702,5 @@
     <inertial>
       <origin
-        xyz="-2.22044604925031E-16 0 0"
+        xyz="2.22044604925031E-16 0 0"
         rpy="0 0 0" />
       <mass
@@ -708,7 +709,7 @@
         ixx="4.97009775274937E-08"
         ixy="-6.61984950467753E-23"
-        ixz="-6.44944990373324E-23"
+        ixz="6.44944990373324E-23"
         iyy="3.95767043274481E-08"
-        iyz="1.03497225198971E-37"
+        iyz="-1.03497225198971E-37"
         izz="3.95767043274481E-08" />
     </inertial>
@@ -742,5 +743,5 @@
     <origin
       xyz="-2.16 -0.26 0.05"
-      rpy="0 0 0" />
+      rpy="0 0 3.1416" />
     <parent
       link="base_link" />
@@ -754,5 +755,5 @@
     <inertial>
       <origin
-        xyz="-2.22044604925031E-16 0 0"
+        xyz="2.22044604925031E-16 0 0"
         rpy="0 0 0" />
       <mass
@@ -761,7 +762,7 @@
         ixx="4.97009775274937E-08"
         ixy="6.61984950467755E-23"
-        ixz="2.20581496680827E-24"
+        ixz="-2.20581496680827E-24"
         iyy="3.95767043274481E-08"
-        iyz="-1.10592535436423E-38"
+        iyz="1.10592535436423E-38"
         izz="3.95767043274481E-08" />
     </inertial>
@@ -795,5 +796,5 @@
     <origin
       xyz="-2.16 -0.6125 0.05"
-      rpy="0 0 0" />
+      rpy="0 0 3.1416" />
     <parent
       link="base_link" />
@@ -807,5 +808,5 @@
     <inertial>
       <origin
-        xyz="0.698189709402004 -5.82219674682042E-17 0.0335520498211091"
+        xyz="-0.698189709402004 5.98392135211463E-17 0.033552049821109"
         rpy="0 0 0" />
       <mass
@@ -813,8 +814,8 @@
       <inertia
         ixx="2433.19483459516"
-        ixy="-2.84228617981465E-13"
-        ixz="-892.315238754295"
+        ixy="-3.12650225766219E-13"
+        ixz="892.315238754295"
         iyy="50275.0478791783"
-        iyz="2.84212143285523E-14"
+        iyz="-2.84212140029952E-14"
         izz="51203.3625667597" />
     </inertial>
@@ -846,5 +847,5 @@
     <origin
       xyz="-2.16 0 0.41495"
-      rpy="0 0 0" />
+      rpy="0 0 3.1416" />
     <parent
       link="base_link" />

File: install/trailer_description/share/trailer_description/urdf/trailer_description.urdf (robot description, URDF)
Before this commit: robot trailer_description, 15 links, 14 joints
Joints:
- joint depth_camera_joint: origin xyz=-2.16 0 0.41495 rpy=0 0 0 -> xyz=-2.16 0 0.41495 rpy=0 0 3.1416
- joint steer_left_joint: limit lower=0 upper=0 effort=100 velocity=31.4 -> lower=-0.6 upper=0.6 effort=50 velocity=31.4
- joint steer_right_joint: limit lower=0 upper=0 effort=100 velocity=31.4 -> lower=-0.6 upper=0.6 effort=50 velocity=31.4
- joint u1_joint: origin xyz=-2.16 0.6125 0.05 rpy=0 0 0 -> xyz=-2.16 0.6125 0.05 rpy=0 0 3.1416
- joint u2_joint: origin xyz=-2.16 0.26 0.05 rpy=0 0 0 -> xyz=-2.16 0.26 0.05 rpy=0 0 3.1416
- joint u3_joint: origin xyz=-2.16 -0.26 0.05 rpy=0 0 0 -> xyz=-2.16 -0.26 0.05 rpy=0 0 3.1416
- joint u4_joint: origin xyz=-2.16 -0.6125 0.05 rpy=0 0 0 -> xyz=-2.16 -0.6125 0.05 rpy=0 0 3.1416

File: install/trailer_description/share/trailer_description/urdf/trailer_gazebo.xacro (robot description, xacro)
@@ -55,4 +55,5 @@
         <maxVel>0.1</maxVel>
         <fdir1>0 1 0</fdir1>
+        <material>Gazebo/Black</material>
     </gazebo>
     <gazebo reference="front_right_wheel">
@@ -64,4 +65,5 @@
         <maxVel>0.1</maxVel>
         <fdir1>0 -1 0</fdir1>
+        <material>Gazebo/Black</material>
     </gazebo>
     <gazebo reference="rear_left_wheel">
@@ -73,4 +75,5 @@
         <maxVel>0.1</maxVel>
         <fdir1>0 1 0</fdir1>
+        <material>Gazebo/Black</material>
     </gazebo>
     <gazebo reference="rear_right_wheel">
@@ -82,4 +85,5 @@
         <maxVel>0.1</maxVel>
         <fdir1>0 -1 0</fdir1>
+        <material>Gazebo/Black</material>
     </gazebo>
     <gazebo reference="trailer">
@@ -91,4 +95,5 @@
         <maxVel>0.1</maxVel>
         <fdir1>0 0 1</fdir1>
+        <material>Gazebo/Blue</material>
     </gazebo>
     <gazebo reference="t_left_wheel">
@@ -100,4 +105,5 @@
         <maxVel>0.1</maxVel>
         <fdir1>0 1 0</fdir1>
+        <material>Gazebo/Black</material>
     </gazebo>
     <gazebo reference="t_right_wheel">
@@ -109,4 +115,23 @@
         <maxVel>0.1</maxVel>
         <fdir1>0 -1 0</fdir1>
+        <material>Gazebo/Black</material>
+    </gazebo>
+    <gazebo>
+        <plugin name="joint_states" filename="libgazebo_ros_joint_state_publisher.so">
+            <ros>
+                <namespace>trailer</namespace>
+                <remapping>~/out:=joint_states</remapping>
+            </ros>
+            <update_rate>30</update_rate>
+            <joint_name>steer_left_joint</joint_name>
+            <joint_name>steer_right_joint</joint_name>
+            <joint_name>front_left_wheel_joint</joint_name>
+            <joint_name>front_right_wheel_joint</joint_name>
+            <joint_name>rear_left_wheel_joint</joint_name>
+            <joint_name>rear_right_wheel_joint</joint_name>
+            <joint_name>trailer_joint</joint_name>
+            <joint_name>t_left_wheel_joint</joint_name>
+            <joint_name>t_right_wheel_joint</joint_name>
+        </plugin>
     </gazebo>
     <gazebo>
@@ -167,14 +192,14 @@
     </gazebo>
     <!-- Ultrasonic Sensor u1 -->
-    <gazebo reference="u1_link">
-        <sensor name="laser_sensor" type="ray">
-            <pose>0 0 0 0 0 0</pose>
+    <gazebo reference="u1_Link">
+        <sensor name="sonar" type="ray">
             <visualize>true</visualize>
             <update_rate>10</update_rate>
+            <always_on>true</always_on>
             <ray>
                 <scan>
                     <horizontal>
                         <samples>10</samples>
-                        <resolution>1</resolution>
+                        <resolution>1.0</resolution>
                         <min_angle>-0.087</min_angle>
                         <max_angle>0.087</max_angle>
@@ -182,5 +207,5 @@
                 </scan>
                 <range>
-                    <min>0.10</min>
+                    <min>0.010</min>
                     <max>8.0</max>
                     <resolution>0.01</resolution>
@@ -196,6 +221,115 @@
                     <remapping>~/out:=range</remapping>
                 </ros>
-                    <topicName>sensor_msgs/Range</topicName>
-                    <frameName>u1_link</frameName>
+                    <output_type>sensor_msgs/Range</output_type>
+                    <topicName>/sensor_msgs/u1_Range</topicName>
+                    <frame_name>u1_Link</frame_name>
+            </plugin>
+        </sensor>
+    </gazebo>
+    <!-- Ultrasonic Sensor u2 -->
+    <gazebo reference="u2_Link">
+        <sensor name="sonar" type="ray">
+            <visualize>true</visualize>
+            <update_rate>10</update_rate>
+            <always_on>true</always_on>
+            <ray>
+                <scan>
+                    <horizontal>
+                        <samples>10</samples>
+                        <resolution>1.0</resolution>
+                        <min_angle>-0.087</min_angle>
+                        <max_angle>0.087</max_angle>
+                    </horizontal>
+                </scan>
+                <range>
+                    <min>0.010</min>
+                    <max>8.0</max>
+                    <resolution>0.01</resolution>
+                </range>
+                <noise>
+                    <type>gaussian</type>
+                    <mean>0.0</mean>
+                    <stddev>0.01</stddev>
+                </noise>
+            </ray>
+            <plugin name="u2_range_sensor" filename="libgazebo_ros_ray_sensor.so">
+                <ros>
+                    <remapping>~/out:=range</remapping>
+                </ros>
+                    <output_type>sensor_msgs/Range</output_type>
+                    <topicName>/sensor_msgs/u2_Range</topicName>
+                    <frame_name>u2_Link</frame_name>
+            </plugin>
+        </sensor>
+    </gazebo>
+    <!-- Ultrasonic Sensor u3 -->
+    <gazebo reference="u3_Link">
+        <sensor name="sonar" type="ray">
+            <visualize>true</visualize>
+            <update_rate>10</update_rate>
+            <always_on>true</always_on>
+            <ray>
+                <scan>
+                    <horizontal>
+                        <samples>10</samples>
+                        <resolution>1.0</resolution>
+                        <min_angle>-0.087</min_angle>
+                        <max_angle>0.087</max_angle>
+                    </horizontal>
+                </scan>
+                <range>
+                    <min>0.010</min>
+                    <max>8.0</max>
+                    <resolution>0.01</resolution>
+                </range>
+                <noise>
+                    <type>gaussian</type>
+                    <mean>0.0</mean>
+                    <stddev>0.01</stddev>
+                </noise>
+            </ray>
+            <plugin name="u3_range_sensor" filename="libgazebo_ros_ray_sensor.so">
+                <ros>
+                    <remapping>~/out:=range</remapping>
+                </ros>
+                    <output_type>sensor_msgs/Range</output_type>
+                    <topicName>/sensor_msgs/u3_Range</topicName>
+                    <frame_name>u3_Link</frame_name>
+            </plugin>
+        </sensor>
+    </gazebo>
+    <!-- Ultrasonic Sensor u4 -->
+    <gazebo reference="u4_Link">
+        <sensor name="sonar" type="ray">
+            <visualize>true</visualize>
+            <update_rate>10</update_rate>
+            <always_on>true</always_on>
+            <ray>
+                <scan>
+                    <horizontal>
+                        <samples>10</samples>
+                        <resolution>1.0</resolution>
+                        <min_angle>-0.087</min_angle>
+                        <max_angle>0.087</max_angle>
+                    </horizontal>
+                </scan>
+                <range>
+                    <min>0.010</min>
+                    <max>8.0</max>
+                    <resolution>0.01</resolution>
+                </range>
+                <noise>
+                    <type>gaussian</type>
+                    <mean>0.0</mean>
+                    <stddev>0.01</stddev>
+                </noise>
+            </ray>
+            <plugin name="u4_range_sensor" filename="libgazebo_ros_ray_sensor.so">
+                <ros>
+                    <remapping>~/out:=range</remapping>
+                </ros>
+                    <output_type>sensor_msgs/Range</output_type>
+                    <topicName>/sensor_msgs/u4_Range</topicName>
+                    <frame_name>u4_Link</frame_name>
             </plugin>
         </sensor>

File: src/trailer_description/urdf/trailer_gazebo.xacro (robot description, xacro)
@@ -55,4 +55,5 @@
         <maxVel>0.1</maxVel>
         <fdir1>0 1 0</fdir1>
+        <material>Gazebo/Black</material>
     </gazebo>
     <gazebo reference="front_right_wheel">
@@ -64,4 +65,5 @@
         <maxVel>0.1</maxVel>
         <fdir1>0 -1 0</fdir1>
+        <material>Gazebo/Black</material>
     </gazebo>
     <gazebo reference="rear_left_wheel">
@@ -73,4 +75,5 @@
         <maxVel>0.1</maxVel>
         <fdir1>0 1 0</fdir1>
+        <material>Gazebo/Black</material>
     </gazebo>
     <gazebo reference="rear_right_wheel">
@@ -82,4 +85,5 @@
         <maxVel>0.1</maxVel>
         <fdir1>0 -1 0</fdir1>
+        <material>Gazebo/Black</material>
     </gazebo>
     <gazebo reference="trailer">
@@ -91,4 +95,5 @@
         <maxVel>0.1</maxVel>
         <fdir1>0 0 1</fdir1>
+        <material>Gazebo/Blue</material>
     </gazebo>
     <gazebo reference="t_left_wheel">
@@ -100,4 +105,5 @@
         <maxVel>0.1</maxVel>
         <fdir1>0 1 0</fdir1>
+        <material>Gazebo/Black</material>
     </gazebo>
     <gazebo reference="t_right_wheel">
@@ -109,4 +115,23 @@
         <maxVel>0.1</maxVel>
         <fdir1>0 -1 0</fdir1>
+        <material>Gazebo/Black</material>
+    </gazebo>
+    <gazebo>
+        <plugin name="joint_states" filename="libgazebo_ros_joint_state_publisher.so">
+            <ros>
+                <namespace>trailer</namespace>
+                <remapping>~/out:=joint_states</remapping>
+            </ros>
+            <update_rate>30</update_rate>
+            <joint_name>steer_left_joint</joint_name>
+            <joint_name>steer_right_joint</joint_name>
+            <joint_name>front_left_wheel_joint</joint_name>
+            <joint_name>front_right_wheel_joint</joint_name>
+            <joint_name>rear_left_wheel_joint</joint_name>
+            <joint_name>rear_right_wheel_joint</joint_name>
+            <joint_name>trailer_joint</joint_name>
+            <joint_name>t_left_wheel_joint</joint_name>
+            <joint_name>t_right_wheel_joint</joint_name>
+        </plugin>
     </gazebo>
     <gazebo>
@@ -167,14 +192,14 @@
     </gazebo>
     <!-- Ultrasonic Sensor u1 -->
-    <gazebo reference="u1_link">
-        <sensor name="laser_sensor" type="ray">
-            <pose>0 0 0 0 0 0</pose>
+    <gazebo reference="u1_Link">
+        <sensor name="sonar" type="ray">
             <visualize>true</visualize>
             <update_rate>10</update_rate>
+            <always_on>true</always_on>
             <ray>
                 <scan>
                     <horizontal>
                         <samples>10</samples>
-                        <resolution>1</resolution>
+                        <resolution>1.0</resolution>
                         <min_angle>-0.087</min_angle>
                         <max_angle>0.087</max_angle>
@@ -182,5 +207,5 @@
                 </scan>
                 <range>
-                    <min>0.10</min>
+                    <min>0.010</min>
                     <max>8.0</max>
                     <resolution>0.01</resolution>
@@ -196,6 +221,111 @@
                     <remapping>~/out:=range</remapping>
                 </ros>
-                    <topicName>sensor_msgs/Range</topicName>
-                    <frameName>u1_link</frameName>
+                    <output_type>sensor_msgs/Range</output_type>
+                    <frame_name>u1_Link</frame_name>
+            </plugin>
+        </sensor>
+    </gazebo>
+    <!-- Ultrasonic Sensor u2 -->
+    <gazebo reference="u2_Link">
+        <sensor name="sonar" type="ray">
+            <visualize>true</visualize>
+            <update_rate>10</update_rate>
+            <always_on>true</always_on>
+            <ray>
+                <scan>
+                    <horizontal>
+                        <samples>10</samples>
+                        <resolution>1.0</resolution>
+                        <min_angle>-0.087</min_angle>
+                        <max_angle>0.087</max_angle>
+                    </horizontal>
+                </scan>
+                <range>
+                    <min>0.010</min>
+                    <max>8.0</max>
+                    <resolution>0.01</resolution>
+                </range>
+                <noise>
+                    <type>gaussian</type>
+                    <mean>0.0</mean>
+                    <stddev>0.01</stddev>
+                </noise>
+            </ray>
+            <plugin name="u2_range_sensor" filename="libgazebo_ros_ray_sensor.so">
+                <ros>
+                    <remapping>~/out:=range</remapping>
+                </ros>
+                    <output_type>sensor_msgs/Range</output_type>
+                    <frame_name>u2_Link</frame_name>
+            </plugin>
+        </sensor>
+    </gazebo>
+    <!-- Ultrasonic Sensor u3 -->
+    <gazebo reference="u3_Link">
+        <sensor name="sonar" type="ray">
+            <visualize>true</visualize>
+            <update_rate>10</update_rate>
+            <always_on>true</always_on>
+            <ray>
+                <scan>
+                    <horizontal>
+                        <samples>10</samples>
+                        <resolution>1.0</resolution>
+                        <min_angle>-0.087</min_angle>
+                        <max_angle>0.087</max_angle>
+                    </horizontal>
+                </scan>
+                <range>
+                    <min>0.010</min>
+                    <max>8.0</max>
+                    <resolution>0.01</resolution>
+                </range>
+                <noise>
+                    <type>gaussian</type>
+                    <mean>0.0</mean>
+                    <stddev>0.01</stddev>
+                </noise>
+            </ray>
+            <plugin name="u3_range_sensor" filename="libgazebo_ros_ray_sensor.so">
+                <ros>
+                    <remapping>~/out:=range</remapping>
+                </ros>
+                    <output_type>sensor_msgs/Range</output_type>
+                    <frame_name>u3_Link</frame_name>
+            </plugin>
+        </sensor>
+    </gazebo>
+    <!-- Ultrasonic Sensor u4 -->
+    <gazebo reference="u4_Link">
+        <sensor name="sonar" type="ray">
+            <visualize>true</visualize>
+            <update_rate>10</update_rate>
+            <always_on>true</always_on>
+            <ray>
+                <scan>
+                    <horizontal>
+                        <samples>10</samples>
+                        <resolution>1.0</resolution>
+                        <min_angle>-0.087</min_angle>
+                        <max_angle>0.087</max_angle>
+                    </horizontal>
+                </scan>
+                <range>
+                    <min>0.010</min>
+                    <max>8.0</max>
+                    <resolution>0.01</resolution>
+                </range>
+                <noise>
+                    <type>gaussian</type>
+                    <mean>0.0</mean>
+                    <stddev>0.01</stddev>
+                </noise>
+            </ray>
+            <plugin name="u4_range_sensor" filename="libgazebo_ros_ray_sensor.so">
+                <ros>
+                    <remapping>~/out:=range</remapping>
+                </ros>
+                    <output_type>sensor_msgs/Range</output_type>
+                    <frame_name>u4_Link</frame_name>
             </plugin>
         </sensor>

Commit message: Few minor changes to trailer_description

File: install/trailer_description/share/trailer_description/urdf/trailer.urdf.xacro (robot description, xacro)
@@ -564,13 +564,4 @@
   <!-- IMU Sensor -->
   <link name="imu_link">
-    <inertial>
-      <mass value="0.01"/>
-      <origin xyz="0.0 0 0" rpy="0 0 0"/>
-      <inertia
-          ixx="1e-7" ixy="0" ixz="0"
-          iyy="1e-7" iyz="0"
-          izz="1e-7"
-      />
-  </inertial>
     <visual>
       <origin xyz="0 0 0" rpy="0 0 0"/>

File: install/trailer_description/share/trailer_description/urdf/trailer_gazebo.xacro (robot description, xacro)
@@ -143,7 +143,8 @@
     </gazebo>
     <gazebo reference="imu_link">
-        <sensor type="imu" name="imu">
+        <sensor type="imu_sensor" name="imu">
             <always_on>true</always_on>
             <update_rate>100</update_rate>
+            <visualize>true</visualize>
             <imu>
                 <angular_velocity>
@@ -188,5 +189,11 @@
                 </linear_acceleration>
             </imu>
-            <plugin filename="libgazebo_ros_imu_sensor.so" name="imu"/>
+            <plugin filename="libgazebo_ros_imu_sensor.so" name="imu">
+                <ros>
+                    <namespace>/trailer</namespace>
+                    <remapping>~/out:=imu</remapping>
+                </ros>
+                <initial_orientation_as_reference>false</initial_orientation_as_reference>
+            </plugin>
         </sensor>
     </gazebo>
