Commit message: Added 5 ArUco markers instead of two

File: install/trailer_description/share/trailer_description/urdf/trailer.urdf.xacro (robot description, xacro)
@@ -563,106 +563,265 @@
   </joint>
   <link
-    name="Left_ArUco_marker">
-    <inertial>
-      <origin
-        xyz="0 0 0"
-        rpy="0 0 0" />
-      <mass
-        value="0.00250000000000084" />
-      <inertia
-        ixx="1.04166666666702E-06"
-        ixy="1.29701920048421E-24"
-        ixz="8.16151537710328E-26"
-        iyy="5.21041666666841E-07"
-        iyz="-2.03287907341201E-23"
-        izz="5.21041666666842E-07" />
-    </inertial>
-    <visual>
-      <origin
-        xyz="0 0 0"
-        rpy="0 0 0" />
-      <geometry>
-        <mesh
-          filename="package://trailer_description/meshes/Left_ArUco_marker.STL" />
-      </geometry>
-      <material
-        name="">
-        <color
-          rgba="0.792156862745098 0.819607843137255 0.933333333333333 1" />
-      </material>
-    </visual>
-    <collision>
-      <origin
-        xyz="0 0 0"
-        rpy="0 0 0" />
-      <geometry>
-        <mesh
-          filename="package://trailer_description/meshes/Left_ArUco_marker.STL" />
-      </geometry>
-    </collision>
-  </link>
-  <joint
-    name="Left_ArUco_joint"
+    name="m1_marker">
+    <inertial>
+      <origin
+        xyz="0 0 2.77555756156289E-17"
+        rpy="0 0 0" />
+      <mass
+        value="0.0100000000000033" />
+      <inertia
+        ixx="1.66666666666723E-05"
+        ixy="4.86161618685412E-24"
+        ixz="-4.86161618685318E-24"
+        iyy="8.33416666666946E-06"
+        iyz="6.38098153595666E-23"
+        izz="8.33416666666947E-06" />
+    </inertial>
+    <visual>
+      <origin
+        xyz="0 0 0"
+        rpy="0 0 0" />
+      <geometry>
+        <mesh
+          filename="package://trailer_description/meshes/m1_marker.STL" />
+      </geometry>
+      <material
+        name="">
+        <color
+          rgba="0.792156862745098 0.819607843137255 0.933333333333333 1" />
+      </material>
+    </visual>
+    <collision>
+      <origin
+        xyz="0 0 0"
+        rpy="0 0 0" />
+      <geometry>
+        <mesh
+          filename="package://trailer_description/meshes/m1_marker.STL" />
+      </geometry>
+    </collision>
+  </link>
+  <joint
+    name="m1_marker_joint"
     type="fixed">
     <origin
-      xyz="-0.84864 0.69 0.55991"
+      xyz="-0.848640000000001 -0.69 0.50991"
       rpy="0 0 0" />
     <parent
       link="trailer" />
     <child
-      link="Left_ArUco_marker" />
+      link="m1_marker" />
     <axis
       xyz="0 0 0" />
   </joint>
   <link
-    name="Right_ArUco_marker">
-    <inertial>
-      <origin
-        xyz="0 0 0"
-        rpy="0 0 0" />
-      <mass
-        value="0.00250000000000084" />
-      <inertia
-        ixx="1.04166666666702E-06"
-        ixy="1.29701920048421E-24"
-        ixz="8.16151537710327E-26"
-        iyy="5.21041666666841E-07"
-        iyz="-2.03287907341201E-23"
-        izz="5.21041666666842E-07" />
-    </inertial>
-    <visual>
-      <origin
-        xyz="0 0 0"
-        rpy="0 0 0" />
-      <geometry>
-        <mesh
-          filename="package://trailer_description/meshes/Right_ArUco_marker.STL" />
-      </geometry>
-      <material
-        name="">
-        <color
-          rgba="0.792156862745098 0.819607843137255 0.933333333333333 1" />
-      </material>
-    </visual>
-    <collision>
-      <origin
-        xyz="0 0 0"
-        rpy="0 0 0" />
-      <geometry>
-        <mesh
-          filename="package://trailer_description/meshes/Right_ArUco_marker.STL" />
-      </geometry>
-    </collision>
-  </link>
-  <joint
-    name="Right_ArUco_joint"
+    name="m2_marker">
+    <inertial>
+      <origin
+        xyz="0 0 1.38777878078145E-17"
+        rpy="0 0 0" />
+      <mass
+        value="0.0100000000000033" />
+      <inertia
+        ixx="1.66666666666722E-05"
+        ixy="-6.52921230174884E-25"
+        ixz="-6.3072190834912E-24"
+        iyy="8.33416666666945E-06"
+        iyz="1.03112144112434E-21"
+        izz="8.33416666666945E-06" />
+    </inertial>
+    <visual>
+      <origin
+        xyz="0 0 0"
+        rpy="0 0 0" />
+      <geometry>
+        <mesh
+          filename="package://trailer_description/meshes/m2_marker.STL" />
+      </geometry>
+      <material
+        name="">
+        <color
+          rgba="0.792156862745098 0.819607843137255 0.933333333333333 1" />
+      </material>
+    </visual>
+    <collision>
+      <origin
+        xyz="0 0 0"
+        rpy="0 0 0" />
+      <geometry>
+        <mesh
+          filename="package://trailer_description/meshes/m2_marker.STL" />
+      </geometry>
+    </collision>
+  </link>
+  <joint
+    name="m2_marker_joint"
     type="fixed">
     <origin
-      xyz="-0.84864 -0.69 0.55991"
+      xyz="-0.848640000000001 -0.345 0.50991"
       rpy="0 0 0" />
     <parent
       link="trailer" />
     <child
-      link="Right_ArUco_marker" />
+      link="m2_marker" />
+    <axis
+      xyz="0 0 0" />
+  </joint>
+  <link
+    name="m3_marker">
+    <inertial>
+      <origin
+        xyz="0 4.79293593203801E-18 1.38777878078145E-17"
+        rpy="0 0 0" />
+      <mass
+        value="0.0100000000000033" />
+      <inertia
+        ixx="1.66666666666722E-05"
+        ixy="-6.52921230175274E-25"
+        ixz="-8.93055070721771E-24"
+        iyy="8.33416666666945E-06"
+        iyz="1.44560289664782E-22"
+        izz="8.33416666666945E-06" />
+    </inertial>
+    <visual>
+      <origin
+        xyz="0 0 0"
+        rpy="0 0 0" />
+      <geometry>
+        <mesh
+          filename="package://trailer_description/meshes/m3_marker.STL" />
+      </geometry>
+      <material
+        name="">
+        <color
+          rgba="0.792156862745098 0.819607843137255 0.933333333333333 1" />
+      </material>
+    </visual>
+    <collision>
+      <origin
+        xyz="0 0 0"
+        rpy="0 0 0" />
+      <geometry>
+        <mesh
+          filename="package://trailer_description/meshes/m3_marker.STL" />
+      </geometry>
+    </collision>
+  </link>
+  <joint
+    name="m3_marker_joint"
+    type="fixed">
+    <origin
+      xyz="-0.84864 0 0.50991"
+      rpy="0 0 0" />
+    <parent
+      link="trailer" />
+    <child
+      link="m3_marker" />
+    <axis
+      xyz="0 0 0" />
+  </joint>
+  <link
+    name="m4_marker">
+    <inertial>
+      <origin
+        xyz="0 5.55111512312578E-17 1.38777878078145E-17"
+        rpy="0 0 0" />
+      <mass
+        value="0.0100000000000033" />
+      <inertia
+        ixx="1.66666666666722E-05"
+        ixy="-6.52921230174884E-25"
+        ixz="-6.3072190834912E-24"
+        iyy="8.33416666666945E-06"
+        iyz="1.03112144112434E-21"
+        izz="8.33416666666945E-06" />
+    </inertial>
+    <visual>
+      <origin
+        xyz="0 0 0"
+        rpy="0 0 0" />
+      <geometry>
+        <mesh
+          filename="package://trailer_description/meshes/m4_marker.STL" />
+      </geometry>
+      <material
+        name="">
+        <color
+          rgba="0.792156862745098 0.819607843137255 0.933333333333333 1" />
+      </material>
+    </visual>
+    <collision>
+      <origin
+        xyz="0 0 0"
+        rpy="0 0 0" />
+      <geometry>
+        <mesh
+          filename="package://trailer_description/meshes/m4_marker.STL" />
+      </geometry>
+    </collision>
+  </link>
+  <joint
+    name="m4_marker_joint"
+    type="fixed">
+    <origin
+      xyz="-0.848640000000001 0.345 0.50991"
+      rpy="0 0 0" />
+    <parent
+      link="trailer" />
+    <child
+      link="m4_marker" />
+    <axis
+      xyz="0 0 0" />
+  </joint>
+  <link
+    name="m5_marker">
+    <inertial>
+      <origin
+        xyz="0 0 2.77555756156289E-17"
+        rpy="0 0 0" />
+      <mass
+        value="0.0100000000000033" />
+      <inertia
+        ixx="1.66666666666723E-05"
+        ixy="4.86161618685412E-24"
+        ixz="-4.86161618685318E-24"
+        iyy="8.33416666666946E-06"
+        iyz="6.38098153595666E-23"
+        izz="8.33416666666947E-06" />
+    </inertial>
+    <visual>
+      <origin
+        xyz="0 0 0"
+        rpy="0 0 0" />
+      <geometry>
+        <mesh
+          filename="package://trailer_description/meshes/m5_marker.STL" />
+      </geometry>
+      <material
+        name="">
+        <color
+          rgba="0.792156862745098 0.819607843137255 0.933333333333333 1" />
+      </material>
+    </visual>
+    <collision>
+      <origin
+        xyz="0 0 0"
+        rpy="0 0 0" />
+      <geometry>
+        <mesh
+          filename="package://trailer_description/meshes/m5_marker.STL" />
+      </geometry>
+    </collision>
+  </link>
+  <joint
+    name="m5_marker_joint"
+    type="fixed">
+    <origin
+      xyz="-0.848640000000001 0.69 0.50991"
+      rpy="0 0 0" />
+    <parent
+      link="trailer" />
+    <child
+      link="m5_marker" />
     <axis
       xyz="0 0 0" />

File: install/trailer_description/share/trailer_description/urdf/trailer_description.urdf (robot description, URDF)
Before this commit: robot trailer_description, 17 links, 16 joints
Links:
- removed link Left_ArUco_marker
- removed link Right_ArUco_marker
- added link m1_marker, mass 0.0100000000000033; collision mesh filename=package://trailer_description/meshes/m1_marker.STL; visual mesh filename=package://trailer_description/meshes/m1_marker.STL
- added link m2_marker, mass 0.0100000000000033; collision mesh filename=package://trailer_description/meshes/m2_marker.STL; visual mesh filename=package://trailer_description/meshes/m2_marker.STL
- added link m3_marker, mass 0.0100000000000033; collision mesh filename=package://trailer_description/meshes/m3_marker.STL; visual mesh filename=package://trailer_description/meshes/m3_marker.STL
- added link m4_marker, mass 0.0100000000000033; collision mesh filename=package://trailer_description/meshes/m4_marker.STL; visual mesh filename=package://trailer_description/meshes/m4_marker.STL
- added link m5_marker, mass 0.0100000000000033; collision mesh filename=package://trailer_description/meshes/m5_marker.STL; visual mesh filename=package://trailer_description/meshes/m5_marker.STL
- link depth_camera_link: mass 8787.20820689569 -> 8787.25320689569
Joints:
- removed joint Left_ArUco_joint
- removed joint Right_ArUco_joint
- added joint m1_marker_joint: type fixed, parent trailer, child m1_marker, origin xyz=-0.848640000000001 -0.69 0.50991 rpy=0 0 0, axis 0 0 0
- added joint m2_marker_joint: type fixed, parent trailer, child m2_marker, origin xyz=-0.848640000000001 -0.345 0.50991 rpy=0 0 0, axis 0 0 0
- added joint m3_marker_joint: type fixed, parent trailer, child m3_marker, origin xyz=-0.84864 0 0.50991 rpy=0 0 0, axis 0 0 0
- added joint m4_marker_joint: type fixed, parent trailer, child m4_marker, origin xyz=-0.848640000000001 0.345 0.50991 rpy=0 0 0, axis 0 0 0
- added joint m5_marker_joint: type fixed, parent trailer, child m5_marker, origin xyz=-0.848640000000001 0.69 0.50991 rpy=0 0 0, axis 0 0 0
- joint steer_left_joint: limit lower=-0.6 upper=0.6 effort=50 velocity=31.4 -> lower=-0.6 upper=0.6 effort=50 velocity=1.5
- joint steer_right_joint: limit lower=-0.6 upper=0.6 effort=50 velocity=31.4 -> lower=-0.6 upper=0.6 effort=50 velocity=1.5
- joint t_left_wheel_joint: axis -0.0225880418212614 -0.999744857634527 0 -> 0.216316683503415 -0.976323252021626 0
- joint t_right_wheel_joint: axis -0.0225880418212613 -0.999744857634527 0 -> 0.216316683503415 -0.976323252021626 0

Commit message: Changed marker mesh to box geometry. Unable to add texture to the marker.

File: install/trailer_description/share/trailer_description/urdf/trailer.urdf.xacro (robot description, xacro)
@@ -583,20 +583,22 @@
         rpy="0 0 0" />
       <geometry>
-        <mesh
-          filename="package://trailer_description/meshes/m1_marker.STL" />
-      </geometry>
-      <material
-        name="">
-        <color
-          rgba="0.792156862745098 0.819607843137255 0.933333333333333 1" />
-      </material>
-    </visual>
-    <collision>
-      <origin
-        xyz="0 0 0"
-        rpy="0 0 0" />
-      <geometry>
-        <mesh
-          filename="package://trailer_description/meshes/m1_marker.STL" />
+        <box size="0.001 0.1 0.1"/>
+      </geometry>
+      <material name="m1_marker_material">
+        <script>
+          <uri>file://trailer_description/materials/textures/m1_marker.png</uri>
+          <name>m1_marker_material</name>
+        </script>
+        <texture>
+          <image filename="package://trailer_description/materials/textures/m1_marker.png"/>
+        </texture>
+      </material>
+    </visual>
+    <collision>
+      <origin
+        xyz="0 0 0"
+        rpy="0 0 0" />
+      <geometry>
+        <box size="0.001 0.1 0.1"/>
       </geometry>
     </collision>
@@ -636,20 +638,18 @@
         rpy="0 0 0" />
       <geometry>
-        <mesh
-          filename="package://trailer_description/meshes/m2_marker.STL" />
-      </geometry>
-      <material
-        name="">
-        <color
-          rgba="0.792156862745098 0.819607843137255 0.933333333333333 1" />
-      </material>
-    </visual>
-    <collision>
-      <origin
-        xyz="0 0 0"
-        rpy="0 0 0" />
-      <geometry>
-        <mesh
-          filename="package://trailer_description/meshes/m2_marker.STL" />
+        <box size="0.001 0.1 0.1"/>
+      </geometry>
+      <material
+        name="">
+        <color
+          rgba="0.792156862745098 0.819607843137255 0.933333333333333 1" />
+      </material>
+    </visual>
+    <collision>
+      <origin
+        xyz="0 0 0"
+        rpy="0 0 0" />
+      <geometry>
+        <box size="0.001 0.1 0.1"/>
       </geometry>
     </collision>
@@ -689,20 +689,18 @@
         rpy="0 0 0" />
       <geometry>
-        <mesh
-          filename="package://trailer_description/meshes/m3_marker.STL" />
-      </geometry>
-      <material
-        name="">
-        <color
-          rgba="0.792156862745098 0.819607843137255 0.933333333333333 1" />
-      </material>
-    </visual>
-    <collision>
-      <origin
-        xyz="0 0 0"
-        rpy="0 0 0" />
-      <geometry>
-        <mesh
-          filename="package://trailer_description/meshes/m3_marker.STL" />
+        <box size="0.001 0.1 0.1"/>
+      </geometry>
+      <material
+        name="">
+        <color
+          rgba="0.792156862745098 0.819607843137255 0.933333333333333 1" />
+      </material>
+    </visual>
+    <collision>
+      <origin
+        xyz="0 0 0"
+        rpy="0 0 0" />
+      <geometry>
+        <box size="0.001 0.1 0.1"/>
       </geometry>
     </collision>
@@ -742,20 +740,18 @@
         rpy="0 0 0" />
       <geometry>
-        <mesh
-          filename="package://trailer_description/meshes/m4_marker.STL" />
-      </geometry>
-      <material
-        name="">
-        <color
-          rgba="0.792156862745098 0.819607843137255 0.933333333333333 1" />
-      </material>
-    </visual>
-    <collision>
-      <origin
-        xyz="0 0 0"
-        rpy="0 0 0" />
-      <geometry>
-        <mesh
-          filename="package://trailer_description/meshes/m4_marker.STL" />
+        <box size="0.001 0.1 0.1"/>
+      </geometry>
+      <material
+        name="">
+        <color
+          rgba="0.792156862745098 0.819607843137255 0.933333333333333 1" />
+      </material>
+    </visual>
+    <collision>
+      <origin
+        xyz="0 0 0"
+        rpy="0 0 0" />
+      <geometry>
+        <box size="0.001 0.1 0.1"/>
       </geometry>
     </collision>
@@ -795,20 +791,18 @@
         rpy="0 0 0" />
       <geometry>
-        <mesh
-          filename="package://trailer_description/meshes/m5_marker.STL" />
-      </geometry>
-      <material
-        name="">
-        <color
-          rgba="0.792156862745098 0.819607843137255 0.933333333333333 1" />
-      </material>
-    </visual>
-    <collision>
-      <origin
-        xyz="0 0 0"
-        rpy="0 0 0" />
-      <geometry>
-        <mesh
-          filename="package://trailer_description/meshes/m5_marker.STL" />
+        <box size="0.001 0.1 0.1"/>
+      </geometry>
+      <material
+        name="">
+        <color
+          rgba="0.792156862745098 0.819607843137255 0.933333333333333 1" />
+      </material>
+    </visual>
+    <collision>
+      <origin
+        xyz="0 0 0"
+        rpy="0 0 0" />
+      <geometry>
+        <box size="0.001 0.1 0.1"/>
       </geometry>
     </collision>

File: src/trailer_description/urdf/trailer.urdf.xacro (robot description, xacro)
@@ -597,6 +597,5 @@
         rpy="0 0 0" />
       <geometry>
-        <mesh
-          filename="package://trailer_description/meshes/m1_marker.STL" />
+        <box size="0.001 0.1 0.1"/>
       </geometry>
     </collision>
@@ -636,20 +635,18 @@
         rpy="0 0 0" />
       <geometry>
-        <mesh
-          filename="package://trailer_description/meshes/m2_marker.STL" />
-      </geometry>
-      <material
-        name="">
-        <color
-          rgba="0.792156862745098 0.819607843137255 0.933333333333333 1" />
-      </material>
-    </visual>
-    <collision>
-      <origin
-        xyz="0 0 0"
-        rpy="0 0 0" />
-      <geometry>
-        <mesh
-          filename="package://trailer_description/meshes/m2_marker.STL" />
+        <box size="0.001 0.1 0.1"/>
+      </geometry>
+      <material
+        name="">
+        <color
+          rgba="0.792156862745098 0.819607843137255 0.933333333333333 1" />
+      </material>
+    </visual>
+    <collision>
+      <origin
+        xyz="0 0 0"
+        rpy="0 0 0" />
+      <geometry>
+        <box size="0.001 0.1 0.1"/>
       </geometry>
     </collision>
@@ -689,20 +686,18 @@
         rpy="0 0 0" />
       <geometry>
-        <mesh
-          filename="package://trailer_description/meshes/m3_marker.STL" />
-      </geometry>
-      <material
-        name="">
-        <color
-          rgba="0.792156862745098 0.819607843137255 0.933333333333333 1" />
-      </material>
-    </visual>
-    <collision>
-      <origin
-        xyz="0 0 0"
-        rpy="0 0 0" />
-      <geometry>
-        <mesh
-          filename="package://trailer_description/meshes/m3_marker.STL" />
+        <box size="0.001 0.1 0.1"/>
+      </geometry>
+      <material
+        name="">
+        <color
+          rgba="0.792156862745098 0.819607843137255 0.933333333333333 1" />
+      </material>
+    </visual>
+    <collision>
+      <origin
+        xyz="0 0 0"
+        rpy="0 0 0" />
+      <geometry>
+        <box size="0.001 0.1 0.1"/>
       </geometry>
     </collision>
@@ -742,20 +737,18 @@
         rpy="0 0 0" />
       <geometry>
-        <mesh
-          filename="package://trailer_description/meshes/m4_marker.STL" />
-      </geometry>
-      <material
-        name="">
-        <color
-          rgba="0.792156862745098 0.819607843137255 0.933333333333333 1" />
-      </material>
-    </visual>
-    <collision>
-      <origin
-        xyz="0 0 0"
-        rpy="0 0 0" />
-      <geometry>
-        <mesh
-          filename="package://trailer_description/meshes/m4_marker.STL" />
+        <box size="0.001 0.1 0.1"/>
+      </geometry>
+      <material
+        name="">
+        <color
+          rgba="0.792156862745098 0.819607843137255 0.933333333333333 1" />
+      </material>
+    </visual>
+    <collision>
+      <origin
+        xyz="0 0 0"
+        rpy="0 0 0" />
+      <geometry>
+        <box size="0.001 0.1 0.1"/>
       </geometry>
     </collision>
@@ -795,20 +788,18 @@
         rpy="0 0 0" />
       <geometry>
-        <mesh
-          filename="package://trailer_description/meshes/m5_marker.STL" />
-      </geometry>
-      <material
-        name="">
-        <color
-          rgba="0.792156862745098 0.819607843137255 0.933333333333333 1" />
-      </material>
-    </visual>
-    <collision>
-      <origin
-        xyz="0 0 0"
-        rpy="0 0 0" />
-      <geometry>
-        <mesh
-          filename="package://trailer_description/meshes/m5_marker.STL" />
+        <box size="0.001 0.1 0.1"/>
+      </geometry>
+      <material
+        name="">
+        <color
+          rgba="0.792156862745098 0.819607843137255 0.933333333333333 1" />
+      </material>
+    </visual>
+    <collision>
+      <origin
+        xyz="0 0 0"
+        rpy="0 0 0" />
+      <geometry>
+        <box size="0.001 0.1 0.1"/>
       </geometry>
     </collision>

Commit message: .

File: install/trailer_description/share/trailer_description/urdf/trailer.urdf.xacro (robot description, xacro)
@@ -583,14 +583,11 @@
         rpy="0 0 0" />
       <geometry>
-        <box size="0.001 0.1 0.1"/>
-      </geometry>
-      <material name="m1_marker_material">
-        <script>
-          <uri>file://trailer_description/materials/textures/m1_marker.png</uri>
-          <name>m1_marker_material</name>
-        </script>
-        <texture>
-          <image filename="package://trailer_description/materials/textures/m1_marker.png"/>
-        </texture>
+        <mesh
+          filename="package://trailer_description/meshes/m1_marker.STL" />
+      </geometry>
+      <material
+        name="">
+        <color
+          rgba="0.792156862745098 0.819607843137255 0.933333333333333 1" />
       </material>
     </visual>

Commit message: ArUco markers are now visible in gazebo. Added the markers to materils script and texture (png file) to /usr/ files

File: install/trailer_description/share/trailer_description/urdf/trailer.urdf.xacro (robot description, xacro)
@@ -583,6 +583,5 @@
         rpy="0 0 0" />
       <geometry>
-        <mesh
-          filename="package://trailer_description/meshes/m1_marker.STL" />
+        <box size="0.001 0.1 0.1"/>
       </geometry>
       <material

File: install/trailer_description/share/trailer_description/urdf/trailer_gazebo.xacro (robot description, xacro)
@@ -142,4 +142,19 @@
         </plugin>
     </gazebo>
+    <gazebo reference="m1_marker">
+        <material>marker/m1_marker</material>
+    </gazebo>
+    <gazebo reference="m2_marker">
+        <material>marker/m2_marker</material>
+    </gazebo>
+    <gazebo reference="m3_marker">
+        <material>marker/m3_marker</material>
+    </gazebo>
+    <gazebo reference="m4_marker">
+        <material>marker/m4_marker</material>
+    </gazebo>
+    <gazebo reference="m5_marker">
+        <material>marker/m5_marker</material>
+    </gazebo>
     <!-- IMU Sensor -->
     <gazebo reference="imu_link">
