Commit message: Performed 5 tests each in 5 scenarios. The files contain the collected data, modified data with range, graphs and their evaluation.

File: install/trailer_description/share/trailer_description/urdf/trailer.urdf.xacro (robot description, xacro)
@@ -583,18 +583,18 @@
         rpy="0 0 0" />
       <geometry>
-        <box size="0.001 0.1 0.1"/>
-      </geometry>
-      <material
-        name="">
-        <color
-          rgba="0.792156862745098 0.819607843137255 0.933333333333333 1" />
-      </material>
-    </visual>
-    <collision>
-      <origin
-        xyz="0 0 0"
-        rpy="0 0 0" />
-      <geometry>
-        <box size="0.001 0.1 0.1"/>
+        <box size="0.001 0.05 0.05"/>
+      </geometry>
+      <material
+        name="">
+        <color
+          rgba="0.792156862745098 0.819607843137255 0.933333333333333 1" />
+      </material>
+    </visual>
+    <collision>
+      <origin
+        xyz="0 0 0"
+        rpy="0 0 0" />
+      <geometry>
+        <box size="0.001 0.05 0.05"/>
       </geometry>
     </collision>
@@ -634,18 +634,18 @@
         rpy="0 0 0" />
       <geometry>
-        <box size="0.001 0.1 0.1"/>
-      </geometry>
-      <material
-        name="">
-        <color
-          rgba="0.792156862745098 0.819607843137255 0.933333333333333 1" />
-      </material>
-    </visual>
-    <collision>
-      <origin
-        xyz="0 0 0"
-        rpy="0 0 0" />
-      <geometry>
-        <box size="0.001 0.1 0.1"/>
+        <box size="0.001 0.05 0.05"/>
+      </geometry>
+      <material
+        name="">
+        <color
+          rgba="0.792156862745098 0.819607843137255 0.933333333333333 1" />
+      </material>
+    </visual>
+    <collision>
+      <origin
+        xyz="0 0 0"
+        rpy="0 0 0" />
+      <geometry>
+        <box size="0.001 0.05 0.05"/>
       </geometry>
     </collision>
@@ -685,18 +685,18 @@
         rpy="0 0 0" />
       <geometry>
-        <box size="0.001 0.1 0.1"/>
-      </geometry>
-      <material
-        name="">
-        <color
-          rgba="0.792156862745098 0.819607843137255 0.933333333333333 1" />
-      </material>
-    </visual>
-    <collision>
-      <origin
-        xyz="0 0 0"
-        rpy="0 0 0" />
-      <geometry>
-        <box size="0.001 0.1 0.1"/>
+        <box size="0.001 0.05 0.05"/>
+      </geometry>
+      <material
+        name="">
+        <color
+          rgba="0.792156862745098 0.819607843137255 0.933333333333333 1" />
+      </material>
+    </visual>
+    <collision>
+      <origin
+        xyz="0 0 0"
+        rpy="0 0 0" />
+      <geometry>
+        <box size="0.001 0.05 0.05"/>
       </geometry>
     </collision>
@@ -736,18 +736,18 @@
         rpy="0 0 0" />
       <geometry>
-        <box size="0.001 0.1 0.1"/>
-      </geometry>
-      <material
-        name="">
-        <color
-          rgba="0.792156862745098 0.819607843137255 0.933333333333333 1" />
-      </material>
-    </visual>
-    <collision>
-      <origin
-        xyz="0 0 0"
-        rpy="0 0 0" />
-      <geometry>
-        <box size="0.001 0.1 0.1"/>
+        <box size="0.001 0.05 0.05"/>
+      </geometry>
+      <material
+        name="">
+        <color
+          rgba="0.792156862745098 0.819607843137255 0.933333333333333 1" />
+      </material>
+    </visual>
+    <collision>
+      <origin
+        xyz="0 0 0"
+        rpy="0 0 0" />
+      <geometry>
+        <box size="0.001 0.05 0.05"/>
       </geometry>
     </collision>
@@ -787,18 +787,18 @@
         rpy="0 0 0" />
       <geometry>
-        <box size="0.001 0.1 0.1"/>
-      </geometry>
-      <material
-        name="">
-        <color
-          rgba="0.792156862745098 0.819607843137255 0.933333333333333 1" />
-      </material>
-    </visual>
-    <collision>
-      <origin
-        xyz="0 0 0"
-        rpy="0 0 0" />
-      <geometry>
-        <box size="0.001 0.1 0.1"/>
+        <box size="0.001 0.05 0.05"/>
+      </geometry>
+      <material
+        name="">
+        <color
+          rgba="0.792156862745098 0.819607843137255 0.933333333333333 1" />
+      </material>
+    </visual>
+    <collision>
+      <origin
+        xyz="0 0 0"
+        rpy="0 0 0" />
+      <geometry>
+        <box size="0.001 0.05 0.05"/>
       </geometry>
     </collision>

Commit message: Added code to mesure the time delay.

File: install/trailer_description/share/trailer_description/urdf/trailer.urdf.xacro (robot description, xacro)
@@ -583,18 +583,18 @@
         rpy="0 0 0" />
       <geometry>
-        <box size="0.001 0.05 0.05"/>
-      </geometry>
-      <material
-        name="">
-        <color
-          rgba="0.792156862745098 0.819607843137255 0.933333333333333 1" />
-      </material>
-    </visual>
-    <collision>
-      <origin
-        xyz="0 0 0"
-        rpy="0 0 0" />
-      <geometry>
-        <box size="0.001 0.05 0.05"/>
+        <box size="0.001 0.1 0.1"/>
+      </geometry>
+      <material
+        name="">
+        <color
+          rgba="0.792156862745098 0.819607843137255 0.933333333333333 1" />
+      </material>
+    </visual>
+    <collision>
+      <origin
+        xyz="0 0 0"
+        rpy="0 0 0" />
+      <geometry>
+        <box size="0.001 0.1 0.1"/>
       </geometry>
     </collision>
@@ -634,18 +634,18 @@
         rpy="0 0 0" />
       <geometry>
-        <box size="0.001 0.05 0.05"/>
-      </geometry>
-      <material
-        name="">
-        <color
-          rgba="0.792156862745098 0.819607843137255 0.933333333333333 1" />
-      </material>
-    </visual>
-    <collision>
-      <origin
-        xyz="0 0 0"
-        rpy="0 0 0" />
-      <geometry>
-        <box size="0.001 0.05 0.05"/>
+        <box size="0.001 0.1 0.1"/>
+      </geometry>
+      <material
+        name="">
+        <color
+          rgba="0.792156862745098 0.819607843137255 0.933333333333333 1" />
+      </material>
+    </visual>
+    <collision>
+      <origin
+        xyz="0 0 0"
+        rpy="0 0 0" />
+      <geometry>
+        <box size="0.001 0.1 0.1"/>
       </geometry>
     </collision>
@@ -685,18 +685,18 @@
         rpy="0 0 0" />
       <geometry>
-        <box size="0.001 0.05 0.05"/>
-      </geometry>
-      <material
-        name="">
-        <color
-          rgba="0.792156862745098 0.819607843137255 0.933333333333333 1" />
-      </material>
-    </visual>
-    <collision>
-      <origin
-        xyz="0 0 0"
-        rpy="0 0 0" />
-      <geometry>
-        <box size="0.001 0.05 0.05"/>
+        <box size="0.001 0.1 0.1"/>
+      </geometry>
+      <material
+        name="">
+        <color
+          rgba="0.792156862745098 0.819607843137255 0.933333333333333 1" />
+      </material>
+    </visual>
+    <collision>
+      <origin
+        xyz="0 0 0"
+        rpy="0 0 0" />
+      <geometry>
+        <box size="0.001 0.1 0.1"/>
       </geometry>
     </collision>
@@ -736,18 +736,18 @@
         rpy="0 0 0" />
       <geometry>
-        <box size="0.001 0.05 0.05"/>
-      </geometry>
-      <material
-        name="">
-        <color
-          rgba="0.792156862745098 0.819607843137255 0.933333333333333 1" />
-      </material>
-    </visual>
-    <collision>
-      <origin
-        xyz="0 0 0"
-        rpy="0 0 0" />
-      <geometry>
-        <box size="0.001 0.05 0.05"/>
+        <box size="0.001 0.1 0.1"/>
+      </geometry>
+      <material
+        name="">
+        <color
+          rgba="0.792156862745098 0.819607843137255 0.933333333333333 1" />
+      </material>
+    </visual>
+    <collision>
+      <origin
+        xyz="0 0 0"
+        rpy="0 0 0" />
+      <geometry>
+        <box size="0.001 0.1 0.1"/>
       </geometry>
     </collision>
@@ -787,18 +787,18 @@
         rpy="0 0 0" />
       <geometry>
-        <box size="0.001 0.05 0.05"/>
-      </geometry>
-      <material
-        name="">
-        <color
-          rgba="0.792156862745098 0.819607843137255 0.933333333333333 1" />
-      </material>
-    </visual>
-    <collision>
-      <origin
-        xyz="0 0 0"
-        rpy="0 0 0" />
-      <geometry>
-        <box size="0.001 0.05 0.05"/>
+        <box size="0.001 0.1 0.1"/>
+      </geometry>
+      <material
+        name="">
+        <color
+          rgba="0.792156862745098 0.819607843137255 0.933333333333333 1" />
+      </material>
+    </visual>
+    <collision>
+      <origin
+        xyz="0 0 0"
+        rpy="0 0 0" />
+      <geometry>
+        <box size="0.001 0.1 0.1"/>
       </geometry>
     </collision>
