Commit message: Updated trailer.urdf.xacro with sensors.

File: src/trailer_description/urdf/trailer.urdf.xacro (robot description, xacro)
@@ -10,5 +10,5 @@
     <inertial>
       <origin
-        xyz="0.0151794504413044 -2.72871741278684E-16 0.504333281484515"
+        xyz="0.0151794504413042 -2.70446273320019E-16 0.504333281484515"
         rpy="0 0 0" />
       <mass
@@ -16,8 +16,8 @@
       <inertia
         ixx="1505.2735842584"
-        ixy="3.7224720704788E-14"
+        ixy="2.45552732709707E-14"
         ixz="-96.1203292275202"
         iyy="7932.64531285603"
-        iyz="-2.22978883011256E-14"
+        iyz="-2.74532801802233E-14"
         izz="8447.43080900142" />
     </inertial>
@@ -161,5 +161,5 @@
     <axis
       xyz="0 1 0" />
-      <limit
+    <limit
       effort="100"
       velocity="31.4" />
@@ -275,5 +275,5 @@
     <axis
       xyz="0 1 0" />
-      <limit
+    <limit
       effort="100"
       velocity="31.4" />
@@ -395,5 +395,5 @@
     <inertial>
       <origin
-        xyz="-2.06473943000056 -9.59060549514745E-17 0.256889099220807"
+        xyz="-2.06473943000056 -9.65449692159716E-17 0.256889099220807"
         rpy="0 0 0" />
       <mass
@@ -401,8 +401,8 @@
       <inertia
         ixx="634.919956534306"
-        ixy="7.66014195843368E-14"
-        ixz="9.29453456945521"
+        ixy="7.7271657034793E-14"
+        ixz="9.29453456945518"
         iyy="1640.30654615615"
-        iyz="4.53164968888437E-15"
+        iyz="4.81260634396325E-15"
         izz="2004.11171155846" />
     </inertial>
@@ -509,5 +509,5 @@
     <inertial>
       <origin
-        xyz="0 0 1.11022302462516E-16"
+        xyz="0 0 0"
         rpy="0 0 0" />
       <mass
@@ -561,4 +561,5 @@
       velocity="31.4" />
   </joint>
+  <!-- IMU Sensor -->
   <link name="imu_link">
     <inertial>
@@ -589,55 +590,267 @@
     <child link="imu_link"/>
   </joint>
-<!-- Ultrasonic Sensors -->
-<xacro:macro name="ultrasonic_sensor" params="name x y z">
-  <link name="${name}">
-    <visual>
-      <origin xyz="${x} ${y} ${z}" rpy="0 0 0"/>
-      <geometry>
-        <cylinder length="0.02" radius="0.015"/>
-      </geometry>
-      <material name="sensor_mat">
-        <color rgba="0.5 0.5 0.5 1"/>
-      </material>
-    </visual>
-  </link>
-  <joint name="${name}_joint" type="fixed">
-    <origin xyz="${x} ${y} ${z}" rpy="0 0 0"/>
-    <parent link="base_link"/>
-    <child link="${name}"/>
-  </joint>
-</xacro:macro>
-<!-- Add Ultrasonic Sensors -->
-<xacro:ultrasonic_sensor name="u1_link" x="-2.16" y="0.6125" z="0.05"/>
-<xacro:ultrasonic_sensor name="u2_link" x="-2.16" y="0.26" z="0.05"/>
-<xacro:ultrasonic_sensor name="u3_link" x="-2.16" y="-0.26" z="0.05"/>
-<xacro:ultrasonic_sensor name="u4_link" x="-2.16" y="-0.6125" z="0.05"/>
-<!-- Depth Sense Camera -->
-<link name="depth_camera_link">
-  <inertial>
-    <origin xyz="0 0 0" rpy="0 0 0"/>
-    <mass value="0.1"/>
-    <inertia ixx="1e-6" ixy="0" ixz="0" iyy="1e-6" iyz="0" izz="1e-6"/>
-  </inertial>
-  <visual>
-    <origin xyz="-2.16 0 0.41495" rpy="0 0 0"/>
-    <geometry>
-      <box size="0.02 0.06 0.015"/>
-    </geometry>
-    <material name="depth_camera_material">
-      <color rgba="0.5 0.5 0.5 1.0"/>
-    </material>
-  </visual>
-  <collision>
-    <origin xyz="-2.16 0 0.41495" rpy="0 0 0"/>
-    <geometry>
-      <box size="0.02 0.06 0.015"/>
-    </geometry>
-  </collision>
-</link>
-<joint name="depth_camera_joint" type="fixed">
-  <origin xyz="-2.16 0 0.41495" rpy="0 0 0"/>
-  <parent link="base_link"/>
-  <child link="depth_camera_link"/>
-</joint>
+  <!-- Ultrasonic Sensors -->
+  <link
+    name="u1_Link">
+    <inertial>
+      <origin
+        xyz="-2.22044604925031E-16 0 0"
+        rpy="0 0 0" />
+      <mass
+        value="0.00176714586764422" />
+      <inertia
+        ixx="4.97009775274937E-08"
+        ixy="6.44944990373328E-23"
+        ixz="1.28060738442034E-40"
+        iyy="3.95767043274481E-08"
+        iyz="-9.95682444457783E-55"
+        izz="3.95767043274481E-08" />
+    </inertial>
+    <visual>
+      <origin
+        xyz="0 0 0"
+        rpy="0 0 0" />
+      <geometry>
+        <mesh
+          filename="package://trailer_description/meshes/u1_Link.STL" />
+      </geometry>
+      <material
+        name="">
+        <color
+          rgba="0.792156862745098 0.819607843137255 0.933333333333333 1" />
+      </material>
+    </visual>
+    <collision>
+      <origin
+        xyz="0 0 0"
+        rpy="0 0 0" />
+      <geometry>
+        <mesh
+          filename="package://trailer_description/meshes/u1_Link.STL" />
+      </geometry>
+    </collision>
+  </link>
+  <joint
+    name="u1_joint"
+    type="fixed">
+    <origin
+      xyz="-2.16 0.6125 0.05"
+      rpy="0 0 0" />
+    <parent
+      link="base_link" />
+    <child
+      link="u1_Link" />
+    <axis
+      xyz="0 0 0" />
+  </joint>
+  <link
+    name="u2_Link">
+    <inertial>
+      <origin
+        xyz="-4.44089209850063E-16 0 0"
+        rpy="0 0 0" />
+      <mass
+        value="0.00176714586764422" />
+      <inertia
+        ixx="4.97009775274937E-08"
+        ixy="-6.61984950467753E-23"
+        ixz="-6.44944990373324E-23"
+        iyy="3.95767043274481E-08"
+        iyz="1.03497225198971E-37"
+        izz="3.95767043274481E-08" />
+    </inertial>
+    <visual>
+      <origin
+        xyz="0 0 0"
+        rpy="0 0 0" />
+      <geometry>
+        <mesh
+          filename="package://trailer_description/meshes/u2_Link.STL" />
+      </geometry>
+      <material
+        name="">
+        <color
+          rgba="0.792156862745098 0.819607843137255 0.933333333333333 1" />
+      </material>
+    </visual>
+    <collision>
+      <origin
+        xyz="0 0 0"
+        rpy="0 0 0" />
+      <geometry>
+        <mesh
+          filename="package://trailer_description/meshes/u2_Link.STL" />
+      </geometry>
+    </collision>
+  </link>
+  <joint
+    name="u2_joint"
+    type="fixed">
+    <origin
+      xyz="-2.16 0.26 0.05"
+      rpy="0 0 0" />
+    <parent
+      link="base_link" />
+    <child
+      link="u2_Link" />
+    <axis
+      xyz="0 0 0" />
+  </joint>
+  <link
+    name="u3_Link">
+    <inertial>
+      <origin
+        xyz="-2.22044604925031E-16 0 0"
+        rpy="0 0 0" />
+      <mass
+        value="0.00176714586764422" />
+      <inertia
+        ixx="4.97009775274937E-08"
+        ixy="-6.61984950467753E-23"
+        ixz="-6.44944990373324E-23"
+        iyy="3.95767043274481E-08"
+        iyz="1.03497225198971E-37"
+        izz="3.95767043274481E-08" />
+    </inertial>
+    <visual>
+      <origin
+        xyz="0 0 0"
+        rpy="0 0 0" />
+      <geometry>
+        <mesh
+          filename="package://trailer_description/meshes/u3_Link.STL" />
+      </geometry>
+      <material
+        name="">
+        <color
+          rgba="0.792156862745098 0.819607843137255 0.933333333333333 1" />
+      </material>
+    </visual>
+    <collision>
+      <origin
+        xyz="0 0 0"
+        rpy="0 0 0" />
+      <geometry>
+        <mesh
+          filename="package://trailer_description/meshes/u3_Link.STL" />
+      </geometry>
+    </collision>
+  </link>
+  <joint
+    name="u3_joint"
+    type="fixed">
+    <origin
+      xyz="-2.16 -0.26 0.05"
+      rpy="0 0 0" />
+    <parent
+      link="base_link" />
+    <child
+      link="u3_Link" />
+    <axis
+      xyz="0 0 0" />
+  </joint>
+  <link
+    name="u4_Link">
+    <inertial>
+      <origin
+        xyz="-2.22044604925031E-16 0 0"
+        rpy="0 0 0" />
+      <mass
+        value="0.00176714586764422" />
+      <inertia
+        ixx="4.97009775274937E-08"
+        ixy="6.61984950467755E-23"
+        ixz="2.20581496680827E-24"
+        iyy="3.95767043274481E-08"
+        iyz="-1.10592535436423E-38"
+        izz="3.95767043274481E-08" />
+    </inertial>
+    <visual>
+      <origin
+        xyz="0 0 0"
+        rpy="0 0 0" />
+      <geometry>
+        <mesh
+          filename="package://trailer_description/meshes/u4_Link.STL" />
+      </geometry>
+      <material
+        name="">
+        <color
+          rgba="0.792156862745098 0.819607843137255 0.933333333333333 1" />
+      </material>
+    </visual>
+    <collision>
+      <origin
+        xyz="0 0 0"
+        rpy="0 0 0" />
+      <geometry>
+        <mesh
+          filename="package://trailer_description/meshes/u4_Link.STL" />
+      </geometry>
+    </collision>
+  </link>
+  <joint
+    name="u4_joint"
+    type="fixed">
+    <origin
+      xyz="-2.16 -0.6125 0.05"
+      rpy="0 0 0" />
+    <parent
+      link="base_link" />
+    <child
+      link="u4_Link" />
+    <axis
+      xyz="0 0 0" />
+  </joint>
+  <link
+    name="depth_camera_link">
+    <inertial>
+      <origin
+        xyz="0.698189709402004 -5.82219674682042E-17 0.0335520498211091"
+        rpy="0 0 0" />
+      <mass
+        value="8787.20320689569" />
+      <inertia
+        ixx="2433.19483459516"
+        ixy="-2.84228617981465E-13"
+        ixz="-892.315238754295"
+        iyy="50275.0478791783"
+        iyz="2.84212143285523E-14"
+        izz="51203.3625667597" />
+    </inertial>
+    <visual>
+      <origin
+        xyz="0 0 0"
+        rpy="0 0 0" />
+      <geometry>
+        <box size="0.02 0.06 0.015"/>
+      </geometry>
+      <material
+        name="">
+        <color
+          rgba="1 1 1 1" />
+      </material>
+    </visual>
+    <collision>
+      <origin
+        xyz="0 0 0"
+        rpy="0 0 0" />
+      <geometry>
+        <box size="0.02 0.06 0.015"/>
+      </geometry>
+    </collision>
+  </link>
+  <joint
+    name="depth_camera_joint"
+    type="fixed">
+    <origin
+      xyz="-2.16 0 0.41495"
+      rpy="0 0 0" />
+    <parent
+      link="base_link" />
+    <child
+      link="depth_camera_link" />
+    <axis
+      xyz="0 0 0" />
+  </joint>
 </robot>

Commit message: Added ArUco Links to the URDF file

File: src/trailer_description/urdf/trailer.urdf.xacro (robot description, xacro)
@@ -562,4 +562,110 @@
       velocity="31.4" />
   </joint>
+  <link
+    name="Left_ArUco_marker">
+    <inertial>
+      <origin
+        xyz="0 0 0"
+        rpy="0 0 0" />
+      <mass
+        value="0.00250000000000084" />
+      <inertia
+        ixx="1.04166666666702E-06"
+        ixy="1.29701920048421E-24"
+        ixz="8.16151537710328E-26"
+        iyy="5.21041666666841E-07"
+        iyz="-2.03287907341201E-23"
+        izz="5.21041666666842E-07" />
+    </inertial>
+    <visual>
+      <origin
+        xyz="0 0 0"
+        rpy="0 0 0" />
+      <geometry>
+        <mesh
+          filename="package://trailer_description/meshes/Left_ArUco_marker.STL" />
+      </geometry>
+      <material
+        name="">
+        <color
+          rgba="0.792156862745098 0.819607843137255 0.933333333333333 1" />
+      </material>
+    </visual>
+    <collision>
+      <origin
+        xyz="0 0 0"
+        rpy="0 0 0" />
+      <geometry>
+        <mesh
+          filename="package://trailer_description/meshes/Left_ArUco_marker.STL" />
+      </geometry>
+    </collision>
+  </link>
+  <joint
+    name="Left_ArUco_joint"
+    type="fixed">
+    <origin
+      xyz="-0.84864 0.69 0.55991"
+      rpy="0 0 0" />
+    <parent
+      link="trailer" />
+    <child
+      link="Left_ArUco_marker" />
+    <axis
+      xyz="0 0 0" />
+  </joint>
+  <link
+    name="Right_ArUco_marker">
+    <inertial>
+      <origin
+        xyz="0 0 0"
+        rpy="0 0 0" />
+      <mass
+        value="0.00250000000000084" />
+      <inertia
+        ixx="1.04166666666702E-06"
+        ixy="1.29701920048421E-24"
+        ixz="8.16151537710327E-26"
+        iyy="5.21041666666841E-07"
+        iyz="-2.03287907341201E-23"
+        izz="5.21041666666842E-07" />
+    </inertial>
+    <visual>
+      <origin
+        xyz="0 0 0"
+        rpy="0 0 0" />
+      <geometry>
+        <mesh
+          filename="package://trailer_description/meshes/Right_ArUco_marker.STL" />
+      </geometry>
+      <material
+        name="">
+        <color
+          rgba="0.792156862745098 0.819607843137255 0.933333333333333 1" />
+      </material>
+    </visual>
+    <collision>
+      <origin
+        xyz="0 0 0"
+        rpy="0 0 0" />
+      <geometry>
+        <mesh
+          filename="package://trailer_description/meshes/Right_ArUco_marker.STL" />
+      </geometry>
+    </collision>
+  </link>
+  <joint
+    name="Right_ArUco_joint"
+    type="fixed">
+    <origin
+      xyz="-0.84864 -0.69 0.55991"
+      rpy="0 0 0" />
+    <parent
+      link="trailer" />
+    <child
+      link="Right_ArUco_marker" />
+    <axis
+      xyz="0 0 0" />
+  </joint>
   <!-- IMU Sensor -->
   <link name="imu_link">

File: src/trailer_description/urdf/trailer_description.urdf (robot description, URDF)
Before this commit: robot trailer_description, 15 links, 14 joints
Links:
- added link Left_ArUco_marker, mass 0.00250000000000084; collision mesh filename=package://trailer_description/meshes/Left_ArUco_marker.STL; visual mesh filename=package://trailer_description/meshes/Left_ArUco_marker.STL
- added link Right_ArUco_marker, mass 0.00250000000000084; collision mesh filename=package://trailer_description/meshes/Right_ArUco_marker.STL; visual mesh filename=package://trailer_description/meshes/Right_ArUco_marker.STL
- link depth_camera_link: mass 8787.20320689569 -> 8787.20820689569
Joints:
- added joint Left_ArUco_joint: type fixed, parent trailer, child Left_ArUco_marker, origin xyz=-0.84864 0.69 0.55991 rpy=0 0 0, axis 0 0 0
- added joint Right_ArUco_joint: type fixed, parent trailer, child Right_ArUco_marker, origin xyz=-0.84864 -0.69 0.55991 rpy=0 0 0, axis 0 0 0
- joint depth_camera_joint: origin xyz=-2.16 0 0.41495 rpy=0 0 3.1416 -> xyz=-2.16 0 0.414953113963299 rpy=0 0 3.14159265358979
- joint rear_left_wheel_joint: origin xyz=-1.17 0.6125 0 rpy=0 0 0 -> xyz=-1.17000000000001 0.612499999999998 0 rpy=0 0 0
- joint rear_right_wheel_joint: origin xyz=-1.17 -0.6125 0 rpy=0 0 0 -> xyz=-1.17000000000001 -0.612499999999998 0 rpy=0 0 0
- joint t_left_wheel_joint: axis 0 -1 0 -> -0.0225880418212614 -0.999744857634527 0; origin xyz=-2.2086 0.6125 -0.15 rpy=0 0 0 -> xyz=-2.20864 0.6125 -0.15 rpy=0 0 0
- joint t_right_wheel_joint: axis 0 -1 0 -> -0.0225880418212613 -0.999744857634527 0; origin xyz=-2.2086 -0.6125 -0.15 rpy=0 0 0 -> xyz=-2.20864 -0.6125 -0.15 rpy=0 0 0

Commit message: Created a dummy link for the depth camera to fix the orientation of the correct point cloud.

File: src/trailer_description/urdf/trailer.urdf.xacro (robot description, xacro)
@@ -1051,5 +1051,5 @@
   </joint>
   <link
-    name="depth_camera_link">
+    name="camera_link">
     <inertial>
       <origin
@@ -1089,5 +1089,5 @@
   </link>
   <joint
-    name="depth_camera_joint"
+    name="camera_joint"
     type="fixed">
     <origin
@@ -1097,7 +1097,13 @@
       link="base_link" />
     <child
-      link="depth_camera_link" />
+      link="camera_link" />
     <axis
       xyz="0 0 0" />
   </joint>
+  <link name="depth_camera_link"/>
+  <joint name="depth_camera_joint" type="fixed">
+      <parent link="camera_link"/>
+      <child link="depth_camera_link"/>
+      <origin xyz="0 0 0" rpy="-1.5708 0 -1.5708"/>
+  </joint>
 </robot>
