Commit message: Added transmission to trailer_gazebo.xacro

File: src/trailer_description/urdf/trailer_gazebo.xacro (robot description, xacro)
@@ -1,4 +1,18 @@
 <?xml version="1.0" encoding="utf-8"?>
 <robot name="trailer" xmlns:xacro="http://www.ros.org/wiki/xacro">
+    <transmission name="left_wheel_transmission">
+        <plugin>transmission_interface/SimpleTransmission</plugin>
+        <actuator name="left_wheel_motor" role="actuator_left"/>
+        <joint name="b_back_left_wheel_joint" role="joint_left">
+            <mechanicalReduction>1.0</mechanicalReduction>
+        </joint>
+    </transmission>
+    <transmission name="right_wheel_transmission">
+        <plugin>transmission_interface/SimpleTransmission</plugin>
+        <actuator name="right_wheel_motor" role="actuator_right"/>
+        <joint name="b_back_right_wheel_joint" role="joint_right">
+            <mechanicalReduction>1.0</mechanicalReduction>
+        </joint>
+    </transmission>
     <gazebo reference="b_front_left_wheel">
         <mu1>100000000000000.0</mu1>
@@ -55,3 +69,10 @@
         <fdir1>0 -1 0</fdir1>
     </gazebo>
+    <gazebo>
+        <plugin filename="libgazebo_ros2_control.so" name="gazebo_ros2_control">
+            <robot_param>robot_description</robot_param>
+            <robot_param_node>robot_state_publisher</robot_param_node>
+            <parameters></parameters>
+        </plugin>
+    </gazebo>
 </robot>

Commit message: Few minor changes to link colors in gazebo and added radiation type for ultrasonic sensors and added vertical element to those sensors.

File: src/trailer_description/urdf/trailer_gazebo.xacro (robot description, xacro)
@@ -95,5 +95,5 @@
         <maxVel>0.1</maxVel>
         <fdir1>0 0 1</fdir1>
-        <material>Gazebo/Blue</material>
+        <material>Gazebo/Orange</material>
     </gazebo>
     <gazebo reference="t_left_wheel">
@@ -200,4 +200,5 @@
     <!-- Ultrasonic Sensor u1 -->
     <gazebo reference="u1_Link">
+        <material>Gazebo/Red</material>
         <sensor name="sonar" type="ray">
             <visualize>true</visualize>
@@ -212,4 +213,10 @@
                         <max_angle>0.087</max_angle>
                     </horizontal>
+                    <vertical>
+                        <samples>10</samples>
+                        <resolution>1.0</resolution>
+                        <min_angle>-0.087</min_angle>
+                        <max_angle>0.087</max_angle>
+                    </vertical>
                 </scan>
                 <range>
@@ -229,4 +236,5 @@
                 </ros>
                     <output_type>sensor_msgs/Range</output_type>
+                    <radiation_type>ultrasound</radiation_type>
                     <frame_name>u1_Link</frame_name>
             </plugin>
@@ -235,4 +243,5 @@
     <!-- Ultrasonic Sensor u2 -->
     <gazebo reference="u2_Link">
+        <material>Gazebo/Red</material>
         <sensor name="sonar" type="ray">
             <visualize>true</visualize>
@@ -247,4 +256,10 @@
                         <max_angle>0.087</max_angle>
                     </horizontal>
+                    <vertical>
+                        <samples>10</samples>
+                        <resolution>1.0</resolution>
+                        <min_angle>-0.087</min_angle>
+                        <max_angle>0.087</max_angle>
+                    </vertical>
                 </scan>
                 <range>
@@ -264,4 +279,5 @@
                 </ros>
                     <output_type>sensor_msgs/Range</output_type>
+                    <radiation_type>ultrasound</radiation_type>
                     <frame_name>u2_Link</frame_name>
             </plugin>
@@ -270,4 +286,5 @@
     <!-- Ultrasonic Sensor u3 -->
     <gazebo reference="u3_Link">
+        <material>Gazebo/Red</material>
         <sensor name="sonar" type="ray">
             <visualize>true</visualize>
@@ -282,4 +299,10 @@
                         <max_angle>0.087</max_angle>
                     </horizontal>
+                    <vertical>
+                        <samples>10</samples>
+                        <resolution>1.0</resolution>
+                        <min_angle>-0.087</min_angle>
+                        <max_angle>0.087</max_angle>
+                    </vertical>
                 </scan>
                 <range>
@@ -299,4 +322,5 @@
                 </ros>
                     <output_type>sensor_msgs/Range</output_type>
+                    <radiation_type>ultrasound</radiation_type>
                     <frame_name>u3_Link</frame_name>
             </plugin>
@@ -305,4 +329,5 @@
     <!-- Ultrasonic Sensor u4 -->
     <gazebo reference="u4_Link">
+        <material>Gazebo/Red</material>
         <sensor name="sonar" type="ray">
             <visualize>true</visualize>
@@ -317,4 +342,10 @@
                         <max_angle>0.087</max_angle>
                     </horizontal>
+                    <vertical>
+                        <samples>10</samples>
+                        <resolution>1.0</resolution>
+                        <min_angle>-0.087</min_angle>
+                        <max_angle>0.087</max_angle>
+                    </vertical>
                 </scan>
                 <range>
@@ -334,4 +365,5 @@
                 </ros>
                     <output_type>sensor_msgs/Range</output_type>
+                    <radiation_type>ultrasound</radiation_type>
                     <frame_name>u4_Link</frame_name>
             </plugin>
@@ -340,4 +372,5 @@
     <!-- Depth Camera Setup -->
     <gazebo reference="depth_camera_link">
+        <material>Gazebo/Black</material>
         <sensor name="depth_camera" type="depth">
             <visualize>true</visualize>

Commit message: Fixed RGB of the point cloud. Fixed the name of the link for the depth camera. And used the camera_link for camera.

File: src/trailer_description/urdf/trailer_gazebo.xacro (robot description, xacro)
@@ -386,7 +386,7 @@
     </gazebo>
     <!-- Depth Camera Setup -->
-    <gazebo reference="depth_camera_link">
-        <material>Gazebo/Black</material>
-        <sensor name="depth_camera" type="depth">
+    <gazebo reference="camera_link">
+        <material>Gazebo/Black</material>
+        <sensor name="camera" type="depth">
             <visualize>true</visualize>
             <update_rate>30.0</update_rate>
@@ -396,5 +396,5 @@
                 <width>640</width>
                 <height>480</height>
-                <format>R8G8B8</format>
+                <format>B8G8R8</format>
             </image>
             <clip>
@@ -407,5 +407,5 @@
                 <alwaysOn>true</alwaysOn>
                 <updateRate>0.0</updateRate>
-                <frame_name>camera_depth_frame</frame_name>
+                <frame_name>depth_camera_link</frame_name>
                 <pointCloudCutoff>0.5</pointCloudCutoff>
                 <pointCloudCutoffMax>3.0</pointCloudCutoffMax>
